File: pcb/kratos-pcb/ioexpantion.kicad_sch (KiCad schematic)
At the start: 3 parts, among them IC2 SN74HC595N, U3 ULN2803A

Commit message: ### update     - kicad schematic
Parts:
- removed RELAY(1-3)1: Conn_01x03_Pin, symbol Connector:Conn_01x03_Pin
- added FREE_OUTPUT1, RELAYS1: Screw_Terminal_01x03, TerminalBlock_4Ucon:TerminalBlock_4Ucon_1x03_P3.50mm_Horizontal, symbol Connector:Screw_Terminal_01x03
- added J2, J3: Screw_Terminal_01x04, TerminalBlock:TerminalBlock_bornier-4_P5.08mm, symbol Connector:Screw_Terminal_01x04
- added U2: ULN2803A, ULN2803A:ULN2803A, symbol Transistor_Array:ULN2803A
- IC2: footprint SN74HC595N:DIP794W53P254L1930H508Q16N -> DIP794W53P254L1930H508Q16N
- U3: footprint (none) -> ULN2803A:ULN2803A
Connections:
- net +5V: now also IC2.10 (~{SRCLR}), U3.10 (COM), J2.4 (Pin_4), J3.4 (Pin_4), U2.10 (COM)
- net GND: now also IC2.13 (~{OE}), U2.9 (GND)
- net B: now reaches IC2.1 (QB)
- net B: now also U3.7 (I7); no longer U3.2 (I2)
- net at IC2.15 (QA): no longer U3.1 (I1)
- net C: now reaches IC2.2 (QC)
- net C: now also U3.6 (I6); no longer U3.3 (I3)
- net D: now reaches IC2.3 (QD)
- net D: now also U3.5 (I5); no longer U3.4 (I4)
- net E: now reaches IC2.4 (QE)
- net E: now also U3.4 (I4); no longer U3.5 (I5)
- net F: now reaches IC2.5 (QF)
- net F: now also U3.3 (I3); no longer U3.6 (I6)
- net G: now reaches IC2.6 (QG)
- net G: now also U3.2 (I2); no longer U3.7 (I7)
- net A: now reaches U3.8 (I8)
- net A: no longer IC2.7 (QH_1)
- net at U3.11 (O8): now also RELAYS1.3 (Pin_3)
- net at U3.12 (O7): now also RELAYS1.2 (Pin_2)
- net at U3.13 (O6): now also RELAYS1.1 (Pin_1)
- net LOCKER_1: now reaches U3.14 (O5)
- net LOCKER_2: now reaches U3.15 (O4)
- net at U3.16 (O3): now also FREE_OUTPUT1.3 (Pin_3)
- net at U3.17 (O2): now also FREE_OUTPUT1.2 (Pin_2)
- net at U3.18 (O1): now also FREE_OUTPUT1.1 (Pin_1)
- new net: J3.3 (Pin_3), U2.13 (O6)
- new net: J3.2 (Pin_2), U2.14 (O5)
- new net: J3.1 (Pin_1), U2.15 (O4)
- new net: J2.3 (Pin_3), U2.16 (O3)
- new net: J2.2 (Pin_2), U2.17 (O2)
- new net: J2.1 (Pin_1), U2.18 (O1)
- new net BLUE-LED: U2.3 (I3)
- new net BLUE-LED-2: U2.6 (I6)
- new net FAN_PWM: U2.11 (O8)
- new net FAN_PWM_DRIVER: U2.8 (I8)
- new net GREEN-LED: U2.2 (I2)
- new net GREEN-LED-2: U2.5 (I5)
- new net H: IC2.7 (QH_1), U3.1 (I1)
- new net RED-LED: U2.1 (I1)
- new net RED-LED-2: U2.4 (I4)
Other:
- note added: "CURRENT DRIVER 2"
- moved on the sheet: IC2, U3

Commit message: ki
Parts:
- removed FREE_OUTPUT1: Screw_Terminal_01x03, TerminalBlock_4Ucon:TerminalBlock_4Ucon_1x03_P3.50mm_Horizontal, symbol Connector:Screw_Terminal_01x03
- added LEDS1: Screw_Terminal_01x03, TerminalBlock_4Ucon:TerminalBlock_4Ucon_1x03_P3.50mm_Horizontal, symbol Connector:Screw_Terminal_01x03
Connections:
- net LOCKER_1: now also U3.17 (O2); no longer U3.14 (O5)
- net LOCKER_2: now also U3.18 (O1); no longer U3.15 (O4)
- net at U3.16 (O3): now also LEDS1.1 (Pin_1)
- new net: LEDS1.2 (Pin_2), U3.15 (O4)
- new net: LEDS1.3 (Pin_3), U3.14 (O5)
Other:
- moved on the sheet: RELAYS1

Commit message: ### MODIFY
Connections:
- net LOCKER_1: now also IC2.6 (QG); no longer U3.17 (O2)
- net LOCKER_2: now also IC2.7 (QH_1); no longer U3.18 (O1)
- net G: no longer names the net of U3.2 (I2)
- net G: no longer IC2.6 (QG)
- net H: no longer names the net of U3.1 (I1)
- net H: no longer IC2.7 (QH_1)
- no-connect marks 3 -> 7
Changed lines of the file:
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@@
   )
   (no_connect (at 71.12 139.7))
+  (no_connect (at 133.35 64.77))
   (no_connect (at 54.61 59.69))
+  (no_connect (at 113.03 62.23))
+  (no_connect (at 133.35 62.23))
   (no_connect (at 91.44 139.7))
+  (no_connect (at 113.03 64.77))
   (bus_entry (at 87.63 72.39) (size 2.54 2.54)
     (stroke (width 0) (type default))
@@
     (stroke (width 0) (type default))
   )
-  (bus_entry (at 109.22 62.23) (size -2.54 2.54)
+  (bus_entry (at 109.22 44.45) (size -2.54 2.54)
     (stroke (width 0) (type default))
   )
@@
     (stroke (width 0) (type default))
   )
-  (bus_entry (at 109.22 64.77) (size -2.54 2.54)
+  (bus_entry (at 109.22 46.99) (size -2.54 2.54)
     (stroke (width 0) (type default))
   )
@@
     (stroke (width 0) (type default))
   )
-  (bus (pts (xy 106.68 67.31) (xy 106.68 69.85))
+  (bus (pts (xy 106.68 49.53) (xy 106.68 69.85))
     (stroke (width 0) (type default))
   )
@@
     (stroke (width 0) (type default))
   )
-  (wire (pts (xy 133.35 62.23) (xy 139.7 62.23))
-    (stroke (width 0) (type default))
-  )
   (wire (pts (xy 135.89 54.61) (xy 135.89 59.69))
     (stroke (width 0) (type default))
@@
     (stroke (width 0) (type default))
   )
-  (wire (pts (xy 109.22 62.23) (xy 113.03 62.23))
-    (stroke (width 0) (type default))
-  )
   (wire (pts (xy 85.09 77.47) (xy 87.63 77.47))
     (stroke (width 0) (type default))
@@
     (stroke (width 0) (type default))
   )
-  (bus (pts (xy 106.68 64.77) (xy 106.68 67.31))
+  (bus (pts (xy 106.68 46.99) (xy 106.68 49.53))
     (stroke (width 0) (type default))
   )
@@
     (stroke (width 0) (type default))
   )
-  (wire (pts (xy 133.35 64.77) (xy 139.7 64.77))
+  (wire (pts (xy 109.22 44.45) (xy 119.38 44.45))
     (stroke (width 0) (type default))
   )
@@
     (stroke (width 0) (type default))
   )
-  (wire (pts (xy 109.22 64.77) (xy 113.03 64.77))
+  (wire (pts (xy 109.22 46.99) (xy 119.38 46.99))
     (stroke (width 0) (type default))
   )
@@
     (effects (font (size 1.27 1.27)) (justify left bottom))
   )
-  (label "H" (at 109.22 62.23 0) (fields_autoplaced)
+  (label "H" (at 109.22 44.45 0) (fields_autoplaced)
     (effects (font (size 1.27 1.27)) (justify left bottom))
   )
@@
     (effects (font (size 1.27 1.27)) (justify left bottom))
   )
-  (label "G" (at 109.22 64.77 0) (fields_autoplaced)
+  (label "G" (at 109.22 46.99 0) (fields_autoplaced)
     (effects (font (size 1.27 1.27)) (justify left bottom))
   )
@@
     )
   )
-  (global_label "LOCKER_1" (shape input) (at 139.7 64.77 0) (fields_autoplaced)
+  (global_label "LOCKER_2" (shape input) (at 119.38 44.45 0) (fields_autoplaced)
     (effects (font (size 1.27 1.27)) (justify left))
-    (property "Intersheetrefs" "${INTERSHEET_REFS}" (at 152.1799 64.77 0)
+    (property "Intersheetrefs" "${INTERSHEET_REFS}" (at 131.8599 44.45 0)
       (effects (font (size 1.27 1.27)) (justify left) hide)
     )
@@
     )
   )
-  (global_label "LOCKER_2" (shape input) (at 139.7 62.23 0) (fields_autoplaced)
+  (global_label "BLUE-LED-2" (shape input) (at 67.31 137.16 180) (fields_autoplaced)
+    (effects (font (size 1.27 1.27)) (justify right))
+    (property "Intersheetrefs" "${INTERSHEET_REFS}" (at 51.7458 137.16 0)
+      (effects (font (size 1.27 1.27)) (justify right) hide)
+    )
+  )
+  (global_label "GREEN-LED" (shape input) (at 67.31 127 180) (fields_autoplaced)
+    (effects (font (size 1.27 1.27)) (justify right))
+    (property "Intersheetrefs" "${INTERSHEET_REFS}" (at 53.1368 127 0)
+      (effects (font (size 1.27 1.27)) (justify right) hide)
+    )
+  )
+  (global_label "BLUE-LED" (shape input) (at 67.31 129.54 180) (fields_autoplaced)
+    (effects (font (size 1.27 1.27)) (justify right))
+    (property "Intersheetrefs" "${INTERSHEET_REFS}" (at 54.5277 129.54 0)
+      (effects (font (size 1.27 1.27)) (justify right) hide)
+    )
+  )
+  (global_label "RED-LED" (shape input) (at 67.31 124.46 180) (fields_autoplaced)
+    (effects (font (size 1.27 1.27)) (justify right))
+    (property "Intersheetrefs" "${INTERSHEET_REFS}" (at 55.6163 124.46 0)
+      (effects (font (size 1.27 1.27)) (justify right) hide)
+    )
+  )
+  (global_label "GREEN-LED-2" (shape input) (at 67.31 134.62 180) (fields_autoplaced)
+    (effects (font (size 1.27 1.27)) (justify right))
+    (property "Intersheetrefs" "${INTERSHEET_REFS}" (at 50.3549 134.62 0)
+      (effects (font (size 1.27 1.27)) (justify right) hide)
+    )
+  )
+  (global_label "LOCKER_1" (shape input) (at 119.38 46.99 0) (fields_autoplaced)
     (effects (font (size 1.27 1.27)) (justify left))
-    (property "Intersheetrefs" "${INTERSHEET_REFS}" (at 152.1799 62.23 0)
+    (property "Intersheetrefs" "${INTERSHEET_REFS}" (at 131.8599 46.99 0)
       (effects (font (size 1.27 1.27)) (justify left) hide)
     )
   )
-  (global_label "BLUE-LED-2" (shape input) (at 67.31 137.16 180) (fields_autoplaced)
-    (effects (font (size 1.27 1.27)) (justify right))
-    (property "Intersheetrefs" "${INTERSHEET_REFS}" (at 51.7458 137.16 0)
-      (effects (font (size 1.27 1.27)) (justify right) hide)
-    )
-  )
-  (global_label "GREEN-LED" (shape input) (at 67.31 127 180) (fields_autoplaced)
-    (effects (font (size 1.27 1.27)) (justify right))
-    (property "Intersheetrefs" "${INTERSHEET_REFS}" (at 53.1368 127 0)
-      (effects (font (size 1.27 1.27)) (justify right) hide)
-    )
-  )
-  (global_label "BLUE-LED" (shape input) (at 67.31 129.54 180) (fields_autoplaced)
-    (effects (font (size 1.27 1.27)) (justify right))
-    (property "Intersheetrefs" "${INTERSHEET_REFS}" (at 54.5277 129.54 0)
-      (effects (font (size 1.27 1.27)) (justify right) hide)
-    )
-  )
-  (global_label "RED-LED" (shape input) (at 67.31 124.46 180) (fields_autoplaced)
-    (effects (font (size 1.27 1.27)) (justify right))
-    (property "Intersheetrefs" "${INTERSHEET_REFS}" (at 55.6163 124.46 0)
-      (effects (font (size 1.27 1.27)) (justify right) hide)
-    )
-  )
-  (global_label "GREEN-LED-2" (shape input) (at 67.31 134.62 180) (fields_autoplaced)
-    (effects (font (size 1.27 1.27)) (justify right))
-    (property "Intersheetrefs" "${INTERSHEET_REFS}" (at 50.3549 134.62 0)
-      (effects (font (size 1.27 1.27)) (justify right) hide)
-    )
-  )

Commit message: ### added
Parts:
- removed J2, J3: Screw_Terminal_01x04, TerminalBlock:TerminalBlock_bornier-4_P5.08mm, symbol Connector:Screw_Terminal_01x04
- added LED-RGB-1.1, LED-RGB-1.2, LED-RGB-2.1, LED-RGB-2.2: Screw_Terminal_01x02, TerminalBlock:TerminalBlock_bornier-2_P5.08mm, symbol Connector:Screw_Terminal_01x02
Connections:
- net +5V: now also LED-RGB-1.1.1 (Pin_1), LED-RGB-2.1.1 (Pin_1)
- net BLUE-LED: now also U2.6 (I6); no longer U2.3 (I3)
- net BLUE-LED-2: now also U2.3 (I3); no longer U2.6 (I6)
- net GREEN-LED: now also U2.5 (I5); no longer U2.2 (I2)
- net GREEN-LED-2: now also U2.1 (I1); no longer U2.5 (I5)
- net RED-LED: now also U2.4 (I4); no longer U2.1 (I1)
- net RED-LED-2: now also U2.2 (I2); no longer U2.4 (I4)
- net at U2.13 (O6): now also LED-RGB-1.1.2 (Pin_2)
- net at U2.14 (O5): now also LED-RGB-1.2.1 (Pin_1)
- net at U2.15 (O4): now also LED-RGB-1.2.2 (Pin_2)
- net at U2.16 (O3): now also LED-RGB-2.1.2 (Pin_2)
- net at U2.17 (O2): now also LED-RGB-2.2.1 (Pin_1)
- net at U2.18 (O1): now also LED-RGB-2.2.2 (Pin_2)
Changed lines of the file:
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@@
+    )
+  )
+  (global_label "BLUE-LED-2" (shape input) (at 67.31 129.54 180) (fields_autoplaced)
+    (effects (font (size 1.27 1.27)) (justify right))
+    (property "Intersheetrefs" "${INTERSHEET_REFS}" (at 51.7458 129.54 0)
+      (effects (font (size 1.27 1.27)) (justify right) hide)
     )
   )
@@
     )
   )
-  (global_label "BLUE-LED-2" (shape input) (at 67.31 137.16 180) (fields_autoplaced)
-    (effects (font (size 1.27 1.27)) (justify right))
-    (property "Intersheetrefs" "${INTERSHEET_REFS}" (at 51.7458 137.16 0)
-      (effects (font (size 1.27 1.27)) (justify right) hide)
-    )
-  )
-  (global_label "GREEN-LED" (shape input) (at 67.31 127 180) (fields_autoplaced)
-    (effects (font (size 1.27 1.27)) (justify right))
-    (property "Intersheetrefs" "${INTERSHEET_REFS}" (at 53.1368 127 0)
-      (effects (font (size 1.27 1.27)) (justify right) hide)
-    )
-  )
-  (global_label "BLUE-LED" (shape input) (at 67.31 129.54 180) (fields_autoplaced)
-    (effects (font (size 1.27 1.27)) (justify right))
-    (property "Intersheetrefs" "${INTERSHEET_REFS}" (at 54.5277 129.54 0)
-      (effects (font (size 1.27 1.27)) (justify right) hide)
-    )
-  )
-  (global_label "RED-LED" (shape input) (at 67.31 124.46 180) (fields_autoplaced)
-    (effects (font (size 1.27 1.27)) (justify right))
-    (property "Intersheetrefs" "${INTERSHEET_REFS}" (at 55.6163 124.46 0)
-      (effects (font (size 1.27 1.27)) (justify right) hide)
-    )
-  )
-  (global_label "GREEN-LED-2" (shape input) (at 67.31 134.62 180) (fields_autoplaced)
-    (effects (font (size 1.27 1.27)) (justify right))
-    (property "Intersheetrefs" "${INTERSHEET_REFS}" (at 50.3549 134.62 0)
+  (global_label "GREEN-LED" (shape input) (at 67.31 134.62 180) (fields_autoplaced)
+    (effects (font (size 1.27 1.27)) (justify right))
+    (property "Intersheetrefs" "${INTERSHEET_REFS}" (at 53.1368 134.62 0)
+      (effects (font (size 1.27 1.27)) (justify right) hide)
+    )
+  )
+  (global_label "GREEN-LED-2" (shape input) (at 67.31 124.46 180) (fields_autoplaced)
+    (effects (font (size 1.27 1.27)) (justify right))
+    (property "Intersheetrefs" "${INTERSHEET_REFS}" (at 50.3549 124.46 0)
       (effects (font (size 1.27 1.27)) (justify right) hide)
     )
@@
     )
   )
+  (global_label "BLUE-LED" (shape input) (at 67.31 137.16 180) (fields_autoplaced)
+    (effects (font (size 1.27 1.27)) (justify right))
+    (property "Intersheetrefs" "${INTERSHEET_REFS}" (at 54.5277 137.16 0)
+      (effects (font (size 1.27 1.27)) (justify right) hide)
+    )
+  )
   (global_label "DS" (shape input) (at 50.8 72.39 180) (fields_autoplaced)
     (effects (font (size 1.27 1.27)) (justify right))
@@
     )
   )
-  (global_label "RED-LED-2" (shape input) (at 67.31 132.08 180) (fields_autoplaced)
-    (effects (font (size 1.27 1.27)) (justify right))
-    (property "Intersheetrefs" "${INTERSHEET_REFS}" (at 52.8344 132.08 0)
+  (global_label "RED-LED" (shape input) (at 67.31 132.08 180) (fields_autoplaced)
+    (effects (font (size 1.27 1.27)) (justify right))
+    (property "Intersheetrefs" "${INTERSHEET_REFS}" (at 55.6163 132.08 0)
+      (effects (font (size 1.27 1.27)) (justify right) hide)
+    )
+  )
+  (global_label "RED-LED-2" (shape input) (at 67.31 127 180) (fields_autoplaced)
+    (effects (font (size 1.27 1.27)) (justify right))
+    (property "Intersheetrefs" "${INTERSHEET_REFS}" (at 52.8344 127 0)
       (effects (font (size 1.27 1.27)) (justify right) hide)
     )
@@
     )
   )
-  (symbol (lib_id "Connector:Screw_Terminal_01x04") (at 107.95 138.43 0) (unit 1)
-    (in_bom yes) (on_board yes) (dnp no) (fields_autoplaced)
-    (property "Reference" "J3" (at 110.49 138.43 0)
-      (effects (font (size 1.27 1.27)) (justify left))
-    )
-    (property "Value" "Screw_Terminal_01x04" (at 110.49 140.97 0)
-      (effects (font (size 1.27 1.27)) (justify left))
-    )
-    (property "Footprint" "TerminalBlock:TerminalBlock_bornier-4_P5.08mm" (at 107.95 138.43 0)
-      (effects (font (size 1.27 1.27)) hide)
-    )
-    (property "Datasheet" "~" (at 107.95 138.43 0)
-      (effects (font (size 1.27 1.27)) hide)
-    )
-    (pin "2")
-    (pin "4")
-    (pin "3")
-    (pin "1")
-    (instances
-      (project "kratos-pcb"
-        (path "/12f1b997-8c5f-4ef7-b036-7873ddaba48e/69401ded-7866-4ef1-bcb6-bf59d95b35e9"
-          (reference "J3") (unit 1)
-        )
-      )
-    )
-  )
   (symbol (lib_id "power:GND") (at 81.28 151.13 0) (unit 1)
     (in_bom yes) (on_board yes) (dnp no) (fields_autoplaced)
@@
     )
   )
+  (symbol (lib_id "Connector:Screw_Terminal_01x02") (at 107.95 127 0) (mirror x) (unit 1)
+    (in_bom yes) (on_board yes) (dnp no) (fields_autoplaced)
+    (property "Reference" "LED-RGB-2.2" (at 110.49 127 0)
+      (effects (font (size 1.27 1.27)) (justify left))
+    )
+    (property "Value" "Screw_Terminal_01x02" (at 110.49 124.46 0)
+      (effects (font (size 1.27 1.27)) (justify left))
+    )
+    (property "Footprint" "TerminalBlock:TerminalBlock_bornier-2_P5.08mm" (at 107.95 127 0)
+      (effects (font (size 1.27 1.27)) hide)
+    )
+    (property "Datasheet" "~" (at 107.95 127 0)
+      (effects (font (size 1.27 1.27)) hide)
+    )
+    (pin "2")
+    (pin "1")
+    (instances
+      (project "kratos-pcb"
+        (path "/12f1b997-8c5f-4ef7-b036-7873ddaba48e/69401ded-7866-4ef1-bcb6-bf59d95b35e9"
+          (reference "LED-RGB-2.2") (unit 1)
+        )
+      )
+    )
+  )
   (symbol (lib_id "power:+5V") (at 53.34 80.01 180) (unit 1)
     (in_bom yes) (on_board yes) (dnp no) (fields_autoplaced)
@@
     )
   )
-  (symbol (lib_id "Connector:Screw_Terminal_01x04") (at 107.95 127 0) (unit 1)
-    (in_bom yes) (on_board yes) (dnp no) (fields_autoplaced)
-    (property "Reference" "J2" (at 110.49 127 0)
-      (effects (font (size 1.27 1.27)) (justify left))
-    )
-    (property "Value" "Screw_Terminal_01x04" (at 110.49 129.54 0)
-      (effects (font (size 1.27 1.27)) (justify left))
-    )
-    (property "Footprint" "TerminalBlock:TerminalBlock_bornier-4_P5.08mm" (at 107.95 127 0)
-      (effects (font (size 1.27 1.27)) hide)
-    )
-    (property "Datasheet" "~" (at 107.95 127 0)
-      (effects (font (size 1.27 1.27)) hide)
-    )
-    (pin "2")
-    (pin "4")
-    (pin "3")
-    (pin "1")
-    (instances
-      (project "kratos-pcb"
-        (path "/12f1b997-8c5f-4ef7-b036-7873ddaba48e/69401ded-7866-4ef1-bcb6-bf59d95b35e9"
-          (reference "J2") (unit 1)
+  (symbol (lib_id "Connector:Screw_Terminal_01x02") (at 107.95 132.08 0) (mirror x) (unit 1)
+    (in_bom yes) (on_board yes) (dnp no) (fields_autoplaced)
+    (property "Reference" "LED-RGB-2.1" (at 110.49 132.08 0)
+      (effects (font (size 1.27 1.27)) (justify left))
+    )
+    (property "Value" "Screw_Terminal_01x02" (at 110.49 129.54 0)
+      (effects (font (size 1.27 1.27)) (justify left))
+    )
+    (property "Footprint" "TerminalBlock:TerminalBlock_bornier-2_P5.08mm" (at 107.95 132.08 0)
+      (effects (font (size 1.27 1.27)) hide)
+    )
+    (property "Datasheet" "~" (at 107.95 132.08 0)
+      (effects (font (size 1.27 1.27)) hide)
+    )
+    (pin "2")
+    (pin "1")
+    (instances
+      (project "kratos-pcb"
+        (path "/12f1b997-8c5f-4ef7-b036-7873ddaba48e/69401ded-7866-4ef1-bcb6-bf59d95b35e9"
+          (reference "LED-RGB-2.1") (unit 1)
         )
       )
@@
     )
   )
+  (symbol (lib_id "Connector:Screw_Terminal_01x02") (at 107.95 143.51 0) (mirror x) (unit 1)
+    (in_bom yes) (on_board yes) (dnp no) (fields_autoplaced)
+    (property "Reference" "LED-RGB-1.1" (at 110.49 143.51 0)
+      (effects (font (size 1.27 1.27)) (justify left))
+    )
+    (property "Value" "Screw_Terminal_01x02" (at 110.49 140.97 0)
+      (effects (font (size 1.27 1.27)) (justify left))
+    )
+    (property "Footprint" "TerminalBlock:TerminalBlock_bornier-2_P5.08mm" (at 107.95 143.51 0)
+      (effects (font (size 1.27 1.27)) hide)
+    )
+    (property "Datasheet" "~" (at 107.95 143.51 0)
+      (effects (font (size 1.27 1.27)) hide)
+    )
+    (pin "2")
+    (pin "1")
+    (instances
+      (project "kratos-pcb"
+        (path "/12f1b997-8c5f-4ef7-b036-7873ddaba48e/69401ded-7866-4ef1-bcb6-bf59d95b35e9"
+          (reference "LED-RGB-1.1") (unit 1)
+        )
+      )
+    )
+  )
   (symbol (lib_id "power:+5V") (at 100.33 116.84 0) (unit 1)
     (in_bom yes) (on_board yes) (dnp no) (fields_autoplaced)
@@
         )
       )
+    )
+  )
+  (symbol (lib_id "Connector:Screw_Terminal_01x02") (at 107.95 138.43 0) (mirror x) (unit 1)
+    (in_bom yes) (on_board yes) (dnp no) (fields_autoplaced)
+    (property "Reference" "LED-RGB-1.2" (at 110.49 138.43 0)
+      (effects (font (size 1.27 1.27)) (justify left))
+    )
+    (property "Value" "Screw_Terminal_01x02" (at 110.49 135.89 0)
+      (effects (font (size 1.27 1.27)) (justify left))
+    )
+    (property "Footprint" "TerminalBlock:TerminalBlock_bornier-2_P5.08mm" (at 107.95 138.43 0)
+      (effects (font (size 1.27 1.27)) hide)
+    )
+    (property "Datasheet" "~" (at 107.95 138.43 0)
+      (effects (font (size 1.27 1.27)) hide)
+    )
+    (pin "2")
+    (pin "1")
+    (instances
+      (project "kratos-pcb"
+        (path "/12f1b997-8c5f-4ef7-b036-7873ddaba48e/69401ded-7866-4ef1-bcb6-bf59d95b35e9"
+          (reference "LED-RGB-1.2") (unit 1)
+        )
+      )

Commit message: ### added
Parts:
- removed LED-RGB-1.1, LED-RGB-1.2, LED-RGB-2.1, LED-RGB-2.2: Screw_Terminal_01x02, TerminalBlock:TerminalBlock_bornier-2_P5.08mm, symbol Connector:Screw_Terminal_01x02
- added J2, J3: Screw_Terminal_01x04, TerminalBlock:TerminalBlock_bornier-4_P5.08mm, symbol Connector:Screw_Terminal_01x04
Connections:
- net +5V: now also J2.4 (Pin_4), J3.4 (Pin_4)
- net BLUE-LED: now also U2.3 (I3); no longer U2.6 (I6)
- net BLUE-LED-2: now also U2.6 (I6); no longer U2.3 (I3)
- net GREEN-LED: now also U2.2 (I2); no longer U2.5 (I5)
- net GREEN-LED-2: now also U2.5 (I5); no longer U2.1 (I1)
- net RED-LED: now also U2.1 (I1); no longer U2.4 (I4)
- net RED-LED-2: now also U2.4 (I4); no longer U2.2 (I2)
- net at U2.13 (O6): now also J3.3 (Pin_3)
- net at U2.14 (O5): now also J3.2 (Pin_2)
- net at U2.15 (O4): now also J3.1 (Pin_1)
- net at U2.16 (O3): now also J2.3 (Pin_3)
- net at U2.17 (O2): now also J2.2 (Pin_2)
- net at U2.18 (O1): now also J2.1 (Pin_1)

Commit message: ### added
Parts:
- removed J2, J3: Screw_Terminal_01x04, TerminalBlock:TerminalBlock_bornier-4_P5.08mm, symbol Connector:Screw_Terminal_01x04
- added LED-RGB-1.1, LED-RGB-1.2, LED-RGB-2.1, LED-RGB-2.2: Screw_Terminal_01x02, TerminalBlock:TerminalBlock_bornier-2_P5.08mm, symbol Connector:Screw_Terminal_01x02
Connections:
- net +5V: now also LED-RGB-1.1.1 (Pin_1), LED-RGB-2.1.1 (Pin_1)
- net BLUE-LED: now also U2.6 (I6); no longer U2.3 (I3)
- net BLUE-LED-2: now also U2.3 (I3); no longer U2.6 (I6)
- net GREEN-LED: now also U2.5 (I5); no longer U2.2 (I2)
- net GREEN-LED-2: now also U2.1 (I1); no longer U2.5 (I5)
- net RED-LED: now also U2.4 (I4); no longer U2.1 (I1)
- net RED-LED-2: now also U2.2 (I2); no longer U2.4 (I4)
- net at U2.13 (O6): now also LED-RGB-1.1.2 (Pin_2)
- net at U2.14 (O5): now also LED-RGB-1.2.1 (Pin_1)
- net at U2.15 (O4): now also LED-RGB-1.2.2 (Pin_2)
- net at U2.16 (O3): now also LED-RGB-2.1.2 (Pin_2)
- net at U2.17 (O2): now also LED-RGB-2.2.1 (Pin_1)
- net at U2.18 (O1): now also LED-RGB-2.2.2 (Pin_2)
- net at RELAYS1.1 (Pin_1): now also U3.11 (O8); no longer U3.13 (O6)
- net at RELAYS1.3 (Pin_3): now also U3.13 (O6); no longer U3.11 (O8)
- net at LEDS1.1 (Pin_1): now also U3.14 (O5); no longer U3.16 (O3)
- net at LEDS1.3 (Pin_3): now also U3.16 (O3); no longer U3.14 (O5)
