File: pcb/kratos-pcb/ioexpantion.kicad_sch (KiCad schematic)
At the start: 9 parts, among them IC2 SN74HC595N, U2 ULN2803A, U3 ULN2803A

Commit message: ### modify
Connections:
- net A: now also IC2.15 (QA)
Changed lines of the file:
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@@
     (stroke (width 0) (type default))
   )
-  (bus (pts (xy 86.36 87.63) (xy 49.53 87.63))
+  (bus (pts (xy 46.99 78.74) (xy 46.99 87.63))
     (stroke (width 0) (type default))
   )
@@
     (stroke (width 0) (type default))
   )
-  (bus (pts (xy 49.53 87.63) (xy 48.26 86.36))
+  (bus (pts (xy 46.99 78.74) (xy 48.26 77.47))
     (stroke (width 0) (type default))
   )
@@
     (stroke (width 0) (type default))
   )
-  (bus (pts (xy 48.26 77.47) (xy 48.26 86.36))
-    (stroke (width 0) (type default))
-  )
   (bus (pts (xy 93.98 87.63) (xy 90.17 83.82))
     (stroke (width 0) (type default))
@@
     (stroke (width 0) (type default))
   )
+  (bus (pts (xy 46.99 87.63) (xy 86.36 87.63))
+    (stroke (width 0) (type default))
+  )
   (wire (pts (xy 102.87 143.51) (xy 101.6 143.51))
     (stroke (width 0) (type default))
@@
     (effects (font (size 1.27 1.27)) (justify left bottom))
   )
+  (label "A" (at 50.8 74.93 0) (fields_autoplaced)
+    (effects (font (size 1.27 1.27)) (justify left bottom))
+  )
   (label "D" (at 86.36 72.39 0) (fields_autoplaced)
     (effects (font (size 1.27 1.27)) (justify left bottom))
@@
     (effects (font (size 1.27 1.27)) (justify left bottom))
   )
-  (label "A" (at 48.26 77.47 90) (fields_autoplaced)
-    (effects (font (size 1.27 1.27)) (justify left bottom))
-  )
