File: pcb/kratos-pcb/ioexpantion.kicad_sch (KiCad schematic)
At the start: 9 parts, among them IC2 SN74HC595N, U2 ULN2803A, U3 ULN2803A

Commit message: ### Modify
   - schematic
Parts:
- removed LEDS1: Screw_Terminal_01x03, TerminalBlock_4Ucon:TerminalBlock_4Ucon_1x03_P3.50mm_Horizontal, symbol Connector:Screw_Terminal_01x03
- added J2, J3, J4: Conn_01x02_Socket, Connector_PinSocket_2.00mm:PinSocket_1x02_P2.00mm_Vertical, symbol Connector:Conn_01x02_Socket
Connections:
- net GND: now also J2.1 (Pin_1), J3.1 (Pin_1), J4.1 (Pin_1)
- net LOCKER_1: now also IC2.9 (QH_2); no longer IC2.6 (QG)
- net LOCKER_2: now also IC2.6 (QG); no longer IC2.7 (QH_1)
- net at U3.14 (O5): now also J4.2 (Pin_2)
- net at U3.15 (O4): now also J3.2 (Pin_2)
- net at U3.16 (O3): now also J2.2 (Pin_2)
