File: pcb/kratos-pcb/rgb.kicad_sch (KiCad schematic)
At the start: 2 parts, among them J3 Conn_01x05_Pin

Commit message: ### added
Parts:
- removed J3: Conn_01x05_Pin, symbol Connector:Conn_01x05_Pin
Other:
- moved on the sheet: LED-STRIP1
Changed lines of the file:
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@@
 (kicad_sch (version 20230121) (generator eeschema)
   (paper "A4")
-  (wire (pts (xy 38.1 36.83) (xy 50.8 36.83))
+  (wire (pts (xy 40.64 40.64) (xy 53.34 40.64))
     (stroke (width 0) (type default))
   )
-  (wire (pts (xy 44.45 44.45) (xy 50.8 44.45))
+  (wire (pts (xy 46.99 48.26) (xy 53.34 48.26))
     (stroke (width 0) (type default))
   )
-  (wire (pts (xy 44.45 48.26) (xy 44.45 44.45))
+  (wire (pts (xy 46.99 52.07) (xy 46.99 48.26))
     (stroke (width 0) (type default))
   )
-  (wire (pts (xy 39.37 41.91) (xy 50.8 41.91))
+  (wire (pts (xy 41.91 45.72) (xy 53.34 45.72))
     (stroke (width 0) (type default))
   )
-  (wire (pts (xy 40.64 39.37) (xy 50.8 39.37))
+  (wire (pts (xy 43.18 43.18) (xy 53.34 43.18))
     (stroke (width 0) (type default))
   )
-  (text "G" (at 45.72 39.37 0)
+  (text "G" (at 48.26 43.18 0)
     (effects (font (size 1.27 1.27)) (justify left bottom))
   )
-  (text "R" (at 45.72 36.83 0)
+  (text "R" (at 48.26 40.64 0)
     (effects (font (size 1.27 1.27)) (justify left bottom))
   )
-  (text "B" (at 45.72 41.91 0)
+  (text "B" (at 48.26 45.72 0)
     (effects (font (size 1.27 1.27)) (justify left bottom))
   )
-  (global_label "BLUE-LED" (shape input) (at 39.37 41.91 180) (fields_autoplaced)
+  (global_label "BLUE-LED" (shape input) (at 41.91 45.72 180) (fields_autoplaced)
     (effects (font (size 1.27 1.27)) (justify right))
-    (property "Intersheetrefs" "${INTERSHEET_REFS}" (at 26.5877 41.91 0)
+    (property "Intersheetrefs" "${INTERSHEET_REFS}" (at 29.1277 45.72 0)
       (effects (font (size 1.27 1.27)) (justify right) hide)
     )
   )
-  (global_label "GREEN-LED" (shape input) (at 40.64 39.37 180) (fields_autoplaced)
+  (global_label "GREEN-LED" (shape input) (at 43.18 43.18 180) (fields_autoplaced)
     (effects (font (size 1.27 1.27)) (justify right))
-    (property "Intersheetrefs" "${INTERSHEET_REFS}" (at 26.4668 39.37 0)
+    (property "Intersheetrefs" "${INTERSHEET_REFS}" (at 29.0068 43.18 0)
       (effects (font (size 1.27 1.27)) (justify right) hide)
     )
   )
-  (global_label "RED-LED" (shape input) (at 38.1 36.83 180) (fields_autoplaced)
+  (global_label "RED-LED" (shape input) (at 40.64 40.64 180) (fields_autoplaced)
     (effects (font (size 1.27 1.27)) (justify right))
-    (property "Intersheetrefs" "${INTERSHEET_REFS}" (at 26.4063 36.83 0)
+    (property "Intersheetrefs" "${INTERSHEET_REFS}" (at 28.9463 40.64 0)
       (effects (font (size 1.27 1.27)) (justify right) hide)
     )
   )
-  (symbol (lib_id "Connector:Conn_01x05_Pin") (at 52.07 71.12 0) (unit 1)
+  (symbol (lib_id "power:GND") (at 46.99 52.07 0) (unit 1)
     (in_bom yes) (on_board yes) (dnp no) (fields_autoplaced)
-    (property "Reference" "J3" (at 52.705 60.96 0)
+    (property "Reference" "#PWR07" (at 46.99 58.42 0)
+      (effects (font (size 1.27 1.27)) hide)
+    )
+    (property "Value" "GND" (at 46.99 57.15 0)
       (effects (font (size 1.27 1.27)))
     )
-    (property "Value" "Conn_01x05_Pin" (at 52.705 63.5 0)
-      (effects (font (size 1.27 1.27)))
-    )
-    (property "Footprint" "" (at 52.07 71.12 0)
+    (property "Footprint" "" (at 46.99 52.07 0)
       (effects (font (size 1.27 1.27)) hide)
     )
-    (property "Datasheet" "~" (at 52.07 71.12 0)
-      (effects (font (size 1.27 1.27)) hide)
-    )
-    (pin "2")
-    (pin "3")
-    (pin "1")
-    (pin "4")
-    (pin "5")
-    (instances
-      (project "kratos-pcb"
-        (path "/12f1b997-8c5f-4ef7-b036-7873ddaba48e/31c82e21-5a03-40d0-b7df-3b432d5f8d2a"
-          (reference "J3") (unit 1)
-        )
-      )
-    )
-  )
-  (symbol (lib_id "power:GND") (at 44.45 48.26 0) (unit 1)
-    (in_bom yes) (on_board yes) (dnp no) (fields_autoplaced)
-    (property "Reference" "#PWR07" (at 44.45 54.61 0)
-      (effects (font (size 1.27 1.27)) hide)
-    )
-    (property "Value" "GND" (at 44.45 53.34 0)
-      (effects (font (size 1.27 1.27)))
-    )
-    (property "Footprint" "" (at 44.45 48.26 0)
-      (effects (font (size 1.27 1.27)) hide)
-    )
-    (property "Datasheet" "" (at 44.45 48.26 0)
+    (property "Datasheet" "" (at 46.99 52.07 0)
       (effects (font (size 1.27 1.27)) hide)
     )
@@
     )
   )
-  (symbol (lib_id "Connector:Conn_01x04_Socket") (at 55.88 39.37 0) (unit 1)
+  (symbol (lib_id "Connector:Conn_01x04_Socket") (at 58.42 43.18 0) (unit 1)
     (in_bom yes) (on_board yes) (dnp no) (fields_autoplaced)
-    (property "Reference" "LED-STRIP1" (at 57.15 39.37 0)
+    (property "Reference" "LED-STRIP1" (at 59.69 43.18 0)
       (effects (font (size 1.27 1.27)) (justify left))
     )
-    (property "Value" "Conn_01x04_Socket" (at 57.15 41.91 0)
+    (property "Value" "Conn_01x04_Socket" (at 59.69 45.72 0)
       (effects (font (size 1.27 1.27)) (justify left))
     )
-    (property "Footprint" "Connector_PinSocket_2.00mm:PinSocket_1x04_P2.00mm_Vertical" (at 55.88 39.37 0)
+    (property "Footprint" "Connector_PinSocket_2.00mm:PinSocket_1x04_P2.00mm_Vertical" (at 58.42 43.18 0)
       (effects (font (size 1.27 1.27)) hide)
     )
-    (property "Datasheet" "~" (at 55.88 39.37 0)
+    (property "Datasheet" "~" (at 58.42 43.18 0)
       (effects (font (size 1.27 1.27)) hide)
     )

Commit message: ### update     - kicad schematic
Parts:
- removed LED-STRIP1: Conn_01x04_Socket, Connector_PinSocket_2.00mm:PinSocket_1x04_P2.00mm_Vertical, symbol Connector:Conn_01x04_Socket
- added J2, J3: Screw_Terminal_01x04, symbol Connector:Screw_Terminal_01x04
- added U2: ULN2803A, ULN2003:DIP794W56P254L1918H533Q16N, symbol Transistor_Array:ULN2803A
Connections:
- net BLUE-LED: now also U2.3 (I3)
- net GND: now also U2.9 (GND)
- net GREEN-LED: now also U2.2 (I2)
- net RED-LED: now also U2.1 (I1)
- new net: J2.1 (Pin_1), U2.18 (O1)
- new net: J2.2 (Pin_2), U2.17 (O2)
- new net: J2.3 (Pin_3), U2.16 (O3)
- new net: J3.1 (Pin_1), U2.15 (O4)
- new net: J3.2 (Pin_2), U2.14 (O5)
- new net: J3.3 (Pin_3), U2.13 (O6)
- new net +5V: J2.4 (Pin_4), J3.4 (Pin_4), U2.10 (COM)
- new net BLUE-LED-2: U2.6 (I6)
- new net FAN_PWM: U2.12 (O7)
- new net FAN_PWM_DRIVER: U2.8 (I8)
- new net GREEN-LED-2: U2.5 (I5)
- new net RED-LED-2: U2.4 (I4)
Other:
- note removed: "B"
- note removed: "G"
- note removed: "R"
