File: pcb/kratos-pcb/power.kicad_sch (KiCad schematic)
At the start: 6 parts, among them J1 Jack-DC

Commit message: ### added
Parts:
- removed C1: C, Capacitor_THT:C_Disc_D3.0mm_W1.6mm_P2.50mm, symbol Device:C
- removed R3: 10, Resistor_THT:R_Axial_DIN0204_L3.6mm_D1.6mm_P5.08mm_Horizontal, symbol Device:R
- R2: value 660 -> 680
Connections:
- net GND: now also R2.1
Other:
- moved on the sheet: J1, R2

Commit message: ### update     - kicad schematic
Parts:
- removed J1: Jack-DC, Connector_BarrelJack:BarrelJack_Horizontal, symbol Connector:Jack-DC
- added C1: 1uF, Capacitor_THT:C_Disc_D3.0mm_W1.6mm_P2.50mm, symbol Device:C
- added C2: 0.1uF, Capacitor_THT:C_Disc_D3.0mm_W1.6mm_P2.50mm, symbol Device:C
- added J1: Barrel_Jack_Switch_Pin3Ring, Connector_BarrelJack:BarrelJack_Horizontal, symbol Connector:Barrel_Jack_Switch_Pin3Ring
- R1: value 200 -> 240
Connections:
- net +5V: now also C1.1
- net GND: now also C1.2, C2.2, J1.3
- net at VR1.3 (VIN): now also C2.1, J1.1
- no-connect marks 0 -> 1
Changed lines of the file:
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@@
   (junction (at 133.35 76.2) (diameter 0) (color 0 0 0 0)
   )
+  (junction (at 132.08 99.06) (diameter 0) (color 0 0 0 0)
+  )
   (junction (at 176.53 96.52) (diameter 0) (color 0 0 0 0)
   )
-  (wire (pts (xy 127 104.14) (xy 130.81 104.14))
+  (no_connect (at 120.65 101.6))
+  (wire (pts (xy 176.53 104.14) (xy 176.53 107.95))
     (stroke (width 0) (type default))
   )
@@
     (stroke (width 0) (type default))
   )
+  (wire (pts (xy 127 104.14) (xy 127 107.95))
+    (stroke (width 0) (type default))
+  )
   (wire (pts (xy 137.16 96.52) (xy 133.35 96.52))
     (stroke (width 0) (type default))
@@
     (stroke (width 0) (type default))
   )
+  (wire (pts (xy 120.65 104.14) (xy 127 104.14))
+    (stroke (width 0) (type default))
+  )
   (wire (pts (xy 133.35 96.52) (xy 133.35 76.2))
     (stroke (width 0) (type default))
@@
     (stroke (width 0) (type default))
   )
-  (wire (pts (xy 127 99.06) (xy 137.16 99.06))
-    (stroke (width 0) (type default))
-  )
   (wire (pts (xy 128.27 76.2) (xy 133.35 76.2))
     (stroke (width 0) (type default))
   )
-  (wire (pts (xy 130.81 104.14) (xy 130.81 109.22))
+  (wire (pts (xy 132.08 99.06) (xy 137.16 99.06))
     (stroke (width 0) (type default))
   )
@@
     (stroke (width 0) (type default))
   )
+  (wire (pts (xy 132.08 106.68) (xy 132.08 107.95))
+    (stroke (width 0) (type default))
+  )
   (wire (pts (xy 118.11 76.2) (xy 118.11 80.01))
     (stroke (width 0) (type default))
@@
   (wire (pts (xy 120.65 76.2) (xy 118.11 76.2))
     (stroke (width 0) (type default))
+  )
+  (wire (pts (xy 120.65 99.06) (xy 132.08 99.06))
+    (stroke (width 0) (type default))
+  )
+  (symbol (lib_id "power:GND") (at 132.08 107.95 0) (unit 1)
+    (in_bom yes) (on_board yes) (dnp no) (fields_autoplaced)
+    (property "Reference" "#PWR019" (at 132.08 114.3 0)
+      (effects (font (size 1.27 1.27)) hide)
+    )
+    (property "Value" "GND" (at 132.08 113.03 0)
+      (effects (font (size 1.27 1.27)))
+    )
+    (property "Footprint" "" (at 132.08 107.95 0)
+      (effects (font (size 1.27 1.27)) hide)
+    )
+    (property "Datasheet" "" (at 132.08 107.95 0)
+      (effects (font (size 1.27 1.27)) hide)
+    )
+    (pin "1")
+    (instances
+      (project "kratos-pcb"
+        (path "/12f1b997-8c5f-4ef7-b036-7873ddaba48e/170159aa-55fb-4081-b17a-e6a087b2344c"
+          (reference "#PWR019") (unit 1)
+        )
+      )
+    )
   )
   (symbol (lib_id "LM317T:LM317T") (at 154.94 99.06 0) (unit 1)
@@
     )
   )
-  (symbol (lib_id "power:GND") (at 130.81 109.22 0) (unit 1)
-    (in_bom yes) (on_board yes) (dnp no) (fields_autoplaced)
-    (property "Reference" "#PWR04" (at 130.81 115.57 0)
-      (effects (font (size 1.27 1.27)) hide)
-    )
-    (property "Value" "GND" (at 130.81 114.3 0)
-      (effects (font (size 1.27 1.27)))
-    )
-    (property "Footprint" "" (at 130.81 109.22 0)
-      (effects (font (size 1.27 1.27)) hide)
-    )
-    (property "Datasheet" "" (at 130.81 109.22 0)
+  (symbol (lib_id "Device:C") (at 176.53 100.33 0) (unit 1)
+    (in_bom yes) (on_board yes) (dnp no) (fields_autoplaced)
+    (property "Reference" "C1" (at 180.34 99.06 0)
+      (effects (font (size 1.27 1.27)) (justify left))
+    )
+    (property "Value" "1uF" (at 180.34 101.6 0)
+      (effects (font (size 1.27 1.27)) (justify left))
+    )
+    (property "Footprint" "Capacitor_THT:C_Disc_D3.0mm_W1.6mm_P2.50mm" (at 177.4952 104.14 0)
+      (effects (font (size 1.27 1.27)) hide)
+    )
+    (property "Datasheet" "~" (at 176.53 100.33 0)
+      (effects (font (size 1.27 1.27)) hide)
+    )
+    (pin "2")
+    (pin "1")
+    (instances
+      (project "kratos-pcb"
+        (path "/12f1b997-8c5f-4ef7-b036-7873ddaba48e/170159aa-55fb-4081-b17a-e6a087b2344c"
+          (reference "C1") (unit 1)
+        )
+      )
+    )
+  )
+  (symbol (lib_id "power:GND") (at 176.53 107.95 0) (unit 1)
+    (in_bom yes) (on_board yes) (dnp no) (fields_autoplaced)
+    (property "Reference" "#PWR020" (at 176.53 114.3 0)
+      (effects (font (size 1.27 1.27)) hide)
+    )
+    (property "Value" "GND" (at 176.53 113.03 0)
+      (effects (font (size 1.27 1.27)))
+    )
+    (property "Footprint" "" (at 176.53 107.95 0)
+      (effects (font (size 1.27 1.27)) hide)
+    )
+    (property "Datasheet" "" (at 176.53 107.95 0)
+      (effects (font (size 1.27 1.27)) hide)
+    )
+    (pin "1")
+    (instances
+      (project "kratos-pcb"
+        (path "/12f1b997-8c5f-4ef7-b036-7873ddaba48e/170159aa-55fb-4081-b17a-e6a087b2344c"
+          (reference "#PWR020") (unit 1)
+        )
+      )
+    )
+  )
+  (symbol (lib_id "power:GND") (at 127 107.95 0) (unit 1)
+    (in_bom yes) (on_board yes) (dnp no) (fields_autoplaced)
+    (property "Reference" "#PWR04" (at 127 114.3 0)
+      (effects (font (size 1.27 1.27)) hide)
+    )
+    (property "Value" "GND" (at 127 113.03 0)
+      (effects (font (size 1.27 1.27)))
+    )
+    (property "Footprint" "" (at 127 107.95 0)
+      (effects (font (size 1.27 1.27)) hide)
+    )
+    (property "Datasheet" "" (at 127 107.95 0)
       (effects (font (size 1.27 1.27)) hide)
     )
@@
       (effects (font (size 1.27 1.27)))
     )
-    (property "Value" "200" (at 154.94 72.39 90)
+    (property "Value" "240" (at 154.94 72.39 90)
       (effects (font (size 1.27 1.27)))
     )
@@
     )
   )
-  (symbol (lib_id "Connector:Jack-DC") (at 119.38 101.6 0) (unit 1)
-    (in_bom yes) (on_board yes) (dnp no) (fields_autoplaced)
-    (property "Reference" "J1" (at 119.38 92.71 0)
-      (effects (font (size 1.27 1.27)))
-    )
-    (property "Value" "Jack-DC" (at 119.38 95.25 0)
-      (effects (font (size 1.27 1.27)))
-    )
-    (property "Footprint" "Connector_BarrelJack:BarrelJack_Horizontal" (at 120.65 102.616 0)
-      (effects (font (size 1.27 1.27)) hide)
-    )
-    (property "Datasheet" "~" (at 120.65 102.616 0)
-      (effects (font (size 1.27 1.27)) hide)
-    )
-    (pin "1")
-    (pin "2")
+  (symbol (lib_id "Connector:Barrel_Jack_Switch_Pin3Ring") (at 113.03 101.6 0) (unit 1)
+    (in_bom yes) (on_board yes) (dnp no) (fields_autoplaced)
+    (property "Reference" "J1" (at 113.03 92.71 0)
+      (effects (font (size 1.27 1.27)))
+    )
+    (property "Value" "Barrel_Jack_Switch_Pin3Ring" (at 113.03 95.25 0)
+      (effects (font (size 1.27 1.27)))
+    )
+    (property "Footprint" "Connector_BarrelJack:BarrelJack_Horizontal" (at 114.3 102.616 0)
+      (effects (font (size 1.27 1.27)) hide)
+    )
+    (property "Datasheet" "~" (at 114.3 102.616 0)
+      (effects (font (size 1.27 1.27)) hide)
+    )
+    (pin "2")
+    (pin "1")
+    (pin "3")
     (instances
       (project "kratos-pcb"
@@
         )
       )
+    )
+  )
+  (symbol (lib_id "Device:C") (at 132.08 102.87 0) (unit 1)
+    (in_bom yes) (on_board yes) (dnp no) (fields_autoplaced)
+    (property "Reference" "C2" (at 135.89 101.6 0)
+      (effects (font (size 1.27 1.27)) (justify left))
+    )
+    (property "Value" "0.1uF" (at 135.89 104.14 0)
+      (effects (font (size 1.27 1.27)) (justify left))
+    )
+    (property "Footprint" "Capacitor_THT:C_Disc_D3.0mm_W1.6mm_P2.50mm" (at 133.0452 106.68 0)
+      (effects (font (size 1.27 1.27)) hide)
+    )
+    (property "Datasheet" "~" (at 132.08 102.87 0)
+      (effects (font (size 1.27 1.27)) hide)
+    )
+    (pin "1")
+    (pin "2")
+    (instances
+      (project "kratos-pcb"
+        (path "/12f1b997-8c5f-4ef7-b036-7873ddaba48e/170159aa-55fb-4081-b17a-e6a087b2344c"
+          (reference "C2") (unit 1)
+        )
+      )

Commit message: kicad
Parts:
- C1: footprint Capacitor_THT:C_Disc_D3.0mm_W1.6mm_P2.50mm -> Capacitor_THT:CP_Radial_D4.0mm_P1.50mm
Connections:
- net +12V: now reaches C2.1, J1.1, VR1.3 (VIN)
Other:
- moved on the sheet: C1, C2, J1, R1, R2
