File: pcb/kratos-pcb/door_lock.kicad_sch (KiCad schematic)
At the start: 8 parts, among them IC1 SN74HC595N, Q2 2N2222A, Q3 2N2222A, U2 74HC595

Commit message: ### added
Parts:
- removed IC1: SN74HC595N, DIP794W53P254L1930H508Q16N, symbol SN74HC595N:SN74HC595N
- removed U2: 74HC595, symbol 74xx:74HC595

Commit message: ### added
Other:
- moved on the sheet: Q2, Q3, R4, R5, R6, R7

Commit message: ### update     - kicad schematic
Parts:
- added LOCK_1, LOCK_2: Screw_Terminal_01x02, TerminalBlock:TerminalBlock_bornier-2_P5.08mm, symbol Connector:Screw_Terminal_01x02
- R4, R5, R6, R7: footprint (none) -> Resistor_THT:R_Axial_DIN0204_L3.6mm_D1.6mm_P5.08mm_Horizontal
Connections:
- net LOCKER_2: now reaches R6.1
- net LOCKER_1: now reaches R7.1
Other:
- note added: "LOCKER 1"
- note added: "LOCKER 2"
- moved on the sheet: Q2, Q3, R4, R5, R6, R7

Commit message: kicad
Parts:
- removed R4, R5: R, Resistor_THT:R_Axial_DIN0204_L3.6mm_D1.6mm_P5.08mm_Horizontal, symbol Device:R
- R7: value R -> 1k
Connections:
- net GND: now reaches Q3.1
- net GND: now also Q2.1
- net at Q3.3: now also LOCK_1.2 (Pin_2)
- net at Q2.3: now also LOCK_2.2 (Pin_2)
- net +12V: now reaches LOCK_2.1 (Pin_1)
- net +12V: now also LOCK_1.1 (Pin_1)
Other:
- moved on the sheet: LOCK_1, LOCK_2, Q2, Q3, R6, R7

Commit message: ki
Parts:
- R6: value R -> 1K
Other:
- moved on the sheet: LOCK_2, Q2, R6

Commit message: ### Modify
   - schematic
Parts:
- added D1, D2: 1N914, Diode_THT:D_DO-35_SOD27_P7.62mm_Horizontal, symbol Diode:1N914
Connections:
- net +12V: now also D1.1 (K), D2.1 (K)
- net at LOCK_1.2 (Pin_2), Q3.3: now also D1.2 (A)
- net at LOCK_2.2 (Pin_2), Q2.3: now also D2.2 (A)
Changed lines of the file:
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@@
 (kicad_sch (version 20230121) (generator eeschema)
   (paper "A4")
-  (wire (pts (xy 185.42 62.23) (xy 185.42 64.77))
+  (junction (at 185.42 67.31) (diameter 0) (color 0 0 0 0)
+  )
+  (junction (at 95.25 63.5) (diameter 0) (color 0 0 0 0)
+  )
+  (junction (at 95.25 71.12) (diameter 0) (color 0 0 0 0)
+  )
+  (junction (at 185.42 59.69) (diameter 0) (color 0 0 0 0)
+  )
+  (wire (pts (xy 185.42 59.69) (xy 185.42 64.77))
     (stroke (width 0) (type default))
   )
@@
     (stroke (width 0) (type default))
   )
+  (wire (pts (xy 88.9 63.5) (xy 95.25 63.5))
+    (stroke (width 0) (type default))
+  )
   (wire (pts (xy 177.8 73.66) (xy 180.34 73.66))
     (stroke (width 0) (type default))
   )
+  (wire (pts (xy 173.99 59.69) (xy 185.42 59.69))
+    (stroke (width 0) (type default))
+  )
   (wire (pts (xy 163.83 73.66) (xy 170.18 73.66))
     (stroke (width 0) (type default))
   )
+  (wire (pts (xy 88.9 71.12) (xy 95.25 71.12))
+    (stroke (width 0) (type default))
+  )
   (wire (pts (xy 85.09 77.47) (xy 90.17 77.47))
     (stroke (width 0) (type default))
@@
     (stroke (width 0) (type default))
   )
-  (wire (pts (xy 95.25 68.58) (xy 95.25 72.39))
-    (stroke (width 0) (type default))
-  )
-  (wire (pts (xy 95.25 62.23) (xy 95.25 66.04))
+  (wire (pts (xy 95.25 68.58) (xy 95.25 71.12))
+    (stroke (width 0) (type default))
+  )
+  (wire (pts (xy 95.25 62.23) (xy 95.25 63.5))
     (stroke (width 0) (type default))
   )
   (wire (pts (xy 71.12 77.47) (xy 77.47 77.47))
+    (stroke (width 0) (type default))
+  )
+  (wire (pts (xy 95.25 63.5) (xy 95.25 66.04))
+    (stroke (width 0) (type default))
+  )
+  (wire (pts (xy 173.99 67.31) (xy 185.42 67.31))
+    (stroke (width 0) (type default))
+  )
+  (wire (pts (xy 185.42 58.42) (xy 185.42 59.69))
+    (stroke (width 0) (type default))
+  )
+  (wire (pts (xy 95.25 71.12) (xy 95.25 72.39))
     (stroke (width 0) (type default))
   )
@@
     )
   )
+  (symbol (lib_id "Diode:1N914") (at 88.9 67.31 90) (mirror x) (unit 1)
+    (in_bom yes) (on_board yes) (dnp no)
+    (property "Reference" "D1" (at 86.36 66.04 90)
+      (effects (font (size 1.27 1.27)) (justify left))
+    )
+    (property "Value" "1N914" (at 86.36 68.58 90)
+      (effects (font (size 1.27 1.27)) (justify left))
+    )
+    (property "Footprint" "Diode_THT:D_DO-35_SOD27_P7.62mm_Horizontal" (at 93.345 67.31 0)
+      (effects (font (size 1.27 1.27)) hide)
+    )
+    (property "Datasheet" "http://www.vishay.com/docs/85622/1n914.pdf" (at 88.9 67.31 0)
+      (effects (font (size 1.27 1.27)) hide)
+    )
+    (property "Sim.Device" "D" (at 88.9 67.31 0)
+      (effects (font (size 1.27 1.27)) hide)
+    )
+    (property "Sim.Pins" "1=K 2=A" (at 88.9 67.31 0)
+      (effects (font (size 1.27 1.27)) hide)
+    )
+    (pin "2")
+    (pin "1")
+    (instances
+      (project "kratos-pcb"
+        (path "/12f1b997-8c5f-4ef7-b036-7873ddaba48e/bcabd817-9513-4d0c-a70f-0efd675264f1"
+          (reference "D1") (unit 1)
+        )
+      )
+    )
+  )
   (symbol (lib_id "Device:R") (at 81.28 77.47 90) (unit 1)
     (in_bom yes) (on_board yes) (dnp no) (fields_autoplaced)
@@
     )
   )
-  (symbol (lib_id "power:+12V") (at 185.42 62.23 0) (unit 1)
-    (in_bom yes) (on_board yes) (dnp no) (fields_autoplaced)
-    (property "Reference" "#PWR023" (at 185.42 66.04 0)
-      (effects (font (size 1.27 1.27)) hide)
-    )
-    (property "Value" "+12V" (at 185.42 57.15 0)
-      (effects (font (size 1.27 1.27)))
-    )
-    (property "Footprint" "" (at 185.42 62.23 0)
-      (effects (font (size 1.27 1.27)) hide)
-    )
-    (property "Datasheet" "" (at 185.42 62.23 0)
+  (symbol (lib_id "power:+12V") (at 185.42 58.42 0) (unit 1)
+    (in_bom yes) (on_board yes) (dnp no) (fields_autoplaced)
+    (property "Reference" "#PWR023" (at 185.42 62.23 0)
+      (effects (font (size 1.27 1.27)) hide)
+    )
+    (property "Value" "+12V" (at 185.42 53.34 0)
+      (effects (font (size 1.27 1.27)))
+    )
+    (property "Footprint" "" (at 185.42 58.42 0)
+      (effects (font (size 1.27 1.27)) hide)
+    )
+    (property "Datasheet" "" (at 185.42 58.42 0)
       (effects (font (size 1.27 1.27)) hide)
     )
@@
         )
       )
+    )
+  )
+  (symbol (lib_id "Diode:1N914") (at 173.99 63.5 90) (mirror x) (unit 1)
+    (in_bom yes) (on_board yes) (dnp no)
+    (property "Reference" "D2" (at 171.45 62.23 90)
+      (effects (font (size 1.27 1.27)) (justify left))
+    )
+    (property "Value" "1N914" (at 171.45 64.77 90)
+      (effects (font (size 1.27 1.27)) (justify left))
+    )
+    (property "Footprint" "Diode_THT:D_DO-35_SOD27_P7.62mm_Horizontal" (at 178.435 63.5 0)
+      (effects (font (size 1.27 1.27)) hide)
+    )
+    (property "Datasheet" "http://www.vishay.com/docs/85622/1n914.pdf" (at 173.99 63.5 0)
+      (effects (font (size 1.27 1.27)) hide)
+    )
+    (property "Sim.Device" "D" (at 173.99 63.5 0)
+      (effects (font (size 1.27 1.27)) hide)
+    )
+    (property "Sim.Pins" "1=K 2=A" (at 173.99 63.5 0)
+      (effects (font (size 1.27 1.27)) hide)
+    )
+    (pin "2")
+    (pin "1")
+    (instances
+      (project "kratos-pcb"
+        (path "/12f1b997-8c5f-4ef7-b036-7873ddaba48e/bcabd817-9513-4d0c-a70f-0efd675264f1"
+          (reference "D2") (unit 1)
+        )
+      )
