File: pcb/kratos-pcb/kratos-pcb.kicad_pcb (KiCad board)
At the start: 2 copper layers, 29 parts, among them IC2 SN74HC595N, J1 Barrel_Jack_Switch_Pin3Ring, Q2 2N2222A, Q3 2N2222A, SW1 SW_Push, U1 ESP32-DEVKIT-V1, U2 ULN2803A, U3 ULN2803A

Commit message: ### modify
Routing:
- net +5V: track 313.2 -> 314.2 mm
Changed lines of the file:
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@@
   (segment (start 175.768 136.906) (end 185.42 136.906) (width 0.5) (layer "F.Cu") (net 0))
   (segment (start 113.4872 101.9048) (end 109.9326 101.9048) (width 1) (layer "F.Cu") (net 1))
-  (segment (start 123.444 74.582) (end 127.668 70.358) (width 1) (layer "F.Cu") (net 1))
   (segment (start 159.7152 101.9048) (end 180.6448 101.9048) (width 1) (layer "F.Cu") (net 1))
   (segment (start 108.2802 65.3288) (end 108.2802 54.5338) (width 1) (layer "F.Cu") (net 1))
   (segment (start 111.252 51.562) (end 111.252 45.974) (width 1) (layer "F.Cu") (net 1))
+  (segment (start 127.254 85.598) (end 126.492 85.598) (width 1) (layer "F.Cu") (net 1))
   (segment (start 175.9712 79.8068) (end 187.452 68.326) (width 1) (layer "F.Cu") (net 1))
+  (segment (start 125.73 70.358) (end 127.254 70.358) (width 1) (layer "F.Cu") (net 1))
   (segment (start 184.3278 93.0402) (end 180.6448 96.7232) (width 0.8) (layer "F.Cu") (net 1))
   (segment (start 169.672 91.948) (end 173.9392 87.6808) (width 1) (layer "F.Cu") (net 1))
@@
   (segment (start 123.444 91.948) (end 113.4872 101.9048) (width 1) (layer "F.Cu") (net 1))
   (segment (start 169.926 79.248) (end 169.926 58.928) (width 1) (layer "F.Cu") (net 1))
-  (segment (start 127.668 85.598) (end 123.444 89.822) (width 1) (layer "F.Cu") (net 1))
+  (segment (start 126.492 85.598) (end 123.444 88.646) (width 1) (layer "F.Cu") (net 1))
   (segment (start 165.3794 54.3814) (end 158.0642 54.3814) (width 1) (layer "F.Cu") (net 1))
   (segment (start 173.9392 83.2612) (end 169.926 79.248) (width 1) (layer "F.Cu") (net 1))
+  (segment (start 123.444 72.644) (end 125.73 70.358) (width 1) (layer "F.Cu") (net 1))
   (segment (start 180.6448 101.9048) (end 182.8292 104.0892) (width 1) (layer "F.Cu") (net 1))
   (segment (start 189.611 93.0402) (end 184.3278 93.0402) (width 0.8) (layer "F.Cu") (net 1))
-  (segment (start 123.444 89.822) (end 123.444 74.582) (width 1) (layer "F.Cu") (net 1))
+  (segment (start 123.444 89.822) (end 123.444 72.644) (width 1) (layer "F.Cu") (net 1))
   (segment (start 108.2802 54.5338) (end 111.252 51.562) (width 1) (layer "F.Cu") (net 1))
   (segment (start 159.7152 101.9048) (end 169.672 91.948) (width 1) (layer "F.Cu") (net 1))
+  (segment (start 123.444 88.646) (end 123.444 89.822) (width 1) (layer "F.Cu") (net 1))
   (segment (start 169.926 58.928) (end 165.3794 54.3814) (width 1) (layer "F.Cu") (net 1))
   (segment (start 103.4946 57.0126) (end 98.5266 57.0126) (width 1) (layer "B.Cu") (net 1))
@@
     (polygon
       (pts
-        (xy 127.762 85.598)
-        (xy 123.444 80.518)
-        (xy 123.444 89.916)
+        (xy 127.254 85.598)
+        (xy 123.317 81.407)
+        (xy 123.19 89.154)
       )
     )
