File: pcb/kratos-pcb/kratos-pcb.kicad_pcb (KiCad board)
At the start: 2 copper layers, 100 x 100 mm, 36 parts, among them IC2 SN74HC595N, J1 Barrel_Jack_Switch_Pin3Ring, Q2 2N2222A, Q3 2N2222A, SW1 SW_Push, U1 ESP32-DEVKIT-V1, U2 ULN2803A, U3 ULN2803A

Commit message: ### better layout
Parts:
- moved R7 0.33 mm to (154.4, 115.8)
Routing:
- net GND: track 196.2 -> 201.6 mm
- net +5V: track 213.6 -> 214.5 mm
Changed lines of the file:
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@@
   )
   (footprint "Resistor_THT:R_Axial_DIN0204_L3.6mm_D1.6mm_P5.08mm_Horizontal" (layer "F.Cu")
-    (at 154.1018 115.7986 -90)
+    (at 154.432 115.7986 -90)
     (descr "Resistor, Axial_DIN0204 series, Axial, Horizontal, pin pitch=5.08mm, 0.167W, length*diameter=3.6*1.6mm^2, http://cdn-reichelt.de/documents/datenblatt/B400/1_4W%23YAG.pdf")
     (tags "Resistor Axial_DIN0204 series Axial Horizontal pin pitch 5.08mm 0.167W length 3.6mm diameter 1.6mm")
@@
   (segment (start 112.268 61.468) (end 102.982 61.468) (width 0.5) (layer "B.Cu") (net 1))
   (segment (start 118.4656 61.468) (end 112.268 61.468) (width 0.5) (layer "B.Cu") (net 1))
-  (segment (start 173.9392 79.8068) (end 170.434 76.3016) (width 0.5) (layer "B.Cu") (net 1))
   (segment (start 162.052 52.324) (end 165.1 52.324) (width 0.5) (layer "B.Cu") (net 1))
+  (segment (start 170.434 77.724) (end 170.434 57.658) (width 0.5) (layer "B.Cu") (net 1))
   (segment (start 110.9472 101.9048) (end 113.284 99.568) (width 0.5) (layer "B.Cu") (net 1))
   (segment (start 108.2802 65.3288) (end 112.141 61.468) (width 0.5) (layer "B.Cu") (net 1))
@@
   (segment (start 189.611 104.0892) (end 193.04 100.6602) (width 0.5) (layer "B.Cu") (net 1))
   (segment (start 128.016 92.202) (end 128.016 86.2584) (width 0.5) (layer "B.Cu") (net 1))
-  (segment (start 170.434 76.3016) (end 170.434 57.658) (width 0.5) (layer "B.Cu") (net 1))
   (segment (start 193.04 69.596) (end 191.77 68.326) (width 0.5) (layer "B.Cu") (net 1))
   (segment (start 191.77 68.326) (end 189.738 68.326) (width 0.5) (layer "B.Cu") (net 1))
@@
   (segment (start 193.04 90.424) (end 193.04 89.916) (width 0.5) (layer "B.Cu") (net 1))
   (segment (start 189.611 104.0892) (end 187.1472 104.0892) (width 0.5) (layer "B.Cu") (net 1))
+  (segment (start 170.434 57.658) (end 167.64 54.864) (width 0.5) (layer "B.Cu") (net 1))
   (segment (start 193.04 100.6602) (end 193.04 89.916) (width 0.5) (layer "B.Cu") (net 1))
   (segment (start 165.1 52.324) (end 167.64 54.864) (width 0.5) (layer "B.Cu") (net 1))
@@
   (segment (start 167.64 54.864) (end 167.1574 54.3814) (width 0.5) (layer "B.Cu") (net 1))
   (segment (start 167.1574 54.3814) (end 158.0642 54.3814) (width 0.5) (layer "B.Cu") (net 1))
+  (segment (start 172.5168 79.8068) (end 170.434 77.724) (width 0.5) (layer "B.Cu") (net 1))
   (segment (start 103.8098 116.5606) (end 98.933 116.5606) (width 0.5) (layer "B.Cu") (net 1))
+  (segment (start 173.9392 79.8068) (end 172.5168 79.8068) (width 0.5) (layer "B.Cu") (net 1))
   (segment (start 187.1472 104.0892) (end 173.9392 90.8812) (width 0.5) (layer "B.Cu") (net 1))
   (segment (start 102.982 61.468) (end 98.5266 57.0126) (width 0.5) (layer "B.Cu") (net 1))
@@
   (segment (start 127 70.0024) (end 118.4656 61.468) (width 0.5) (layer "B.Cu") (net 1))
   (segment (start 109.9326 101.9048) (end 109.9326 111.8094) (width 0.5) (layer "B.Cu") (net 1))
-  (segment (start 170.434 57.658) (end 167.64 54.864) (width 0.5) (layer "B.Cu") (net 1))
   (segment (start 123.952 73.0504) (end 127 70.0024) (width 0.5) (layer "B.Cu") (net 1))
   (segment (start 105.1814 116.5606) (end 103.8098 116.5606) (width 0.5) (layer "B.Cu") (net 1))
@@
   (segment (start 125.476 128.0668) (end 110.7548 128.0668) (width 0.5) (layer "B.Cu") (net 2))
   (segment (start 132.6642 56.9214) (end 122.1994 56.9214) (width 0.5) (layer "B.Cu") (net 2))
+  (segment (start 115.2906 50.0126) (end 113.0752 47.7972) (width 0.5) (layer "B.Cu") (net 2))
+  (segment (start 113.0752 47.7972) (end 113.0752 45.5676) (width 0.5) (layer "B.Cu") (net 2))
   (segment (start 107.3745 132.89) (end 107.3745 124.6865) (width 0.5) (layer "B.Cu") (net 2))
   (segment (start 108.4326 101.9048) (end 108.4326 98.4098) (width 0.5) (layer "B.Cu") (net 2))
@@
   (segment (start 139.8524 122.3264) (end 139.7 122.174) (width 0.5) (layer "B.Cu") (net 13))
   (segment (start 139.8524 128.0668) (end 139.8524 122.3264) (width 0.5) (layer "B.Cu") (net 13))
+  (segment (start 154.2542 121.031) (end 154.1018 120.8786) (width 0.5) (layer "B.Cu") (net 14))
   (segment (start 154.2542 128.3716) (end 154.2542 121.031) (width 0.5) (layer "B.Cu") (net 14))
-  (segment (start 154.2542 121.031) (end 154.1018 120.8786) (width 0.5) (layer "B.Cu") (net 14))
   (segment (start 98.8314 111.5314) (end 98.8568 111.5568) (width 0.5) (layer "B.Cu") (net 15))
   (segment (start 101.3206 114.0206) (end 103.8098 114.0206) (width 0.5) (layer "B.Cu") (net 15))
@@
   (segment (start 120.2944 85.2424) (end 119.06 85.2424) (width 0.5) (layer "B.Cu") (net 16))
   (segment (start 122.682 87.63) (end 120.2944 85.2424) (width 0.5) (layer "B.Cu") (net 16))
-  (segment (start 149.606 109.22) (end 154.1018 113.7158) (width 0.5) (layer "B.Cu") (net 17))
+  (segment (start 119.06 82.7024) (end 120.5484 82.7024) (width 0.5) (layer "B.Cu") (net 17))
+  (segment (start 121.158 83.375827) (end 124.714 86.931827) (width 0.5) (layer "B.Cu") (net 17))
   (segment (start 124.714 93.472) (end 140.462 109.22) (width 0.5) (layer "B.Cu") (net 17))
   (segment (start 124.714 86.931827) (end 124.714 93.472) (width 0.5) (layer "B.Cu") (net 17))
+  (segment (start 149.606 109.22) (end 154.432 114.046) (width 0.5) (layer "B.Cu") (net 17))
   (segment (start 140.462 109.22) (end 149.606 109.22) (width 0.5) (layer "B.Cu") (net 17))
+  (segment (start 120.5484 82.7024) (end 121.158 83.312) (width 0.5) (layer "B.Cu") (net 17))
   (segment (start 121.158 83.312) (end 121.158 83.375827) (width 0.5) (layer "B.Cu") (net 17))
-  (segment (start 121.158 83.375827) (end 124.714 86.931827) (width 0.5) (layer "B.Cu") (net 17))
-  (segment (start 120.5484 82.7024) (end 121.158 83.312) (width 0.5) (layer "B.Cu") (net 17))
-  (segment (start 154.1018 113.7158) (end 154.1018 115.7986) (width 0.5) (layer "B.Cu") (net 17))
-  (segment (start 119.06 82.7024) (end 120.5484 82.7024) (width 0.5) (layer "B.Cu") (net 17))
+  (segment (start 154.432 114.046) (end 154.432 115.7986) (width 0.5) (layer "B.Cu") (net 17))
   (segment (start 176.784 90.678) (end 185.1152 99.0092) (width 0.5) (layer "B.Cu") (net 18))
   (segment (start 176.784 78.232) (end 176.784 90.678) (width 0.5) (layer "B.Cu") (net 18))
@@
   (segment (start 166.3192 77.2668) (end 158.0896 77.2668) (width 0.5) (layer "B.Cu") (net 39))
   (segment (start 158.0896 77.2668) (end 158.0642 77.2414) (width 0.5) (layer "B.Cu") (net 39))
-  (segment (start 158.0134 89.9414) (end 154.94 86.868) (width 0.5) (layer "B.Cu") (net 40))
+  (segment (start 157.7594 89.9414) (end 154.94 87.122) (width 0.5) (layer "B.Cu") (net 40))
   (segment (start 158.0134 50.2666) (end 170.3094 50.2666) (width 0.5) (layer "B.Cu") (net 40))
   (segment (start 170.3094 50.2666) (end 176.8094 50.2666) (width 0.5) (layer "B.Cu") (net 40))
-  (segment (start 158.0642 89.9414) (end 158.0134 89.9414) (width 0.5) (layer "B.Cu") (net 40))
+  (segment (start 158.0642 89.9414) (end 157.7594 89.9414) (width 0.5) (layer "B.Cu") (net 40))
+  (segment (start 154.94 87.122) (end 154.94 53.34) (width 0.5) (layer "B.Cu") (net 40))
   (segment (start 154.94 53.34) (end 158.0134 50.2666) (width 0.5) (layer "B.Cu") (net 40))
-  (segment (start 154.94 86.868) (end 154.94 53.34) (width 0.5) (layer "B.Cu") (net 40))
   (segment (start 115.9002 80.5688) (end 118.6536 80.5688) (width 0.5) (layer "B.Cu") (net 42))
   (segment (start 118.6536 80.5688) (end 119.06 80.1624) (width 0.5) (layer "B.Cu") (net 42))

Commit message: ### Modify
   - schematic
Parts:
- removed LEDS1: Screw_Terminal_01x03, TerminalBlock_4Ucon:TerminalBlock_4Ucon_1x03_P3.50mm_Horizontal
- removed the REF** at (128.0, 92.2)
- removed the REF** at (162.3, 56.9)
- removed the REF** at (165.1, 45.7)
- removed the REF** at (119.1, 66.0)
- removed the REF** at (170.7, 84.8)
- removed the REF** at (162.1, 52.3)
- removed the REF** at (113.3, 99.6)
- removed SW1: SW_Push, Button_Switch_THT:SW_PUSH_6mm_H4.3mm
- added ?: , , F.Cu at (124.7, 137.7)
- added ?: , , F.Cu at (150.4, 60.7)
- added ?: , , F.Cu at (120.1, 137.7)
- added ?: , , F.Cu at (137.7, 61.7)
- added D1: 1N914, Diode_THT:D_DO-35_SOD27_P7.62mm_Horizontal, F.Cu at (166.9, 138.2)
- added D2: 1N914, Diode_THT:D_DO-35_SOD27_P7.62mm_Horizontal, F.Cu at (131.6, 140.5)
- added J2: Conn_01x02_Socket, Connector_PinSocket_2.00mm:PinSocket_1x02_P2.00mm_Vertical, F.Cu at (98.8, 88.1)
- added J3: Conn_01x02_Socket, Connector_PinSocket_2.00mm:PinSocket_1x02_P2.00mm_Vertical, F.Cu at (98.8, 83.0)
- added J4: Conn_01x02_Socket, Connector_PinSocket_2.00mm:PinSocket_1x02_P2.00mm_Vertical, F.Cu at (98.8, 77.7)
- added R3: 10k, Resistor_THT:R_Axial_DIN0207_L6.3mm_D2.5mm_P10.16mm_Horizontal, F.Cu at (154.4, 107.7)
- added R4: 10k, Resistor_THT:R_Axial_DIN0207_L6.3mm_D2.5mm_P10.16mm_Horizontal, F.Cu at (156.0, 103.6)
- added REF**: SolderWirePad_1x01_SMD_1x2mm, Connector_Wire:SolderWirePad_1x01_SMD_1x2mm, F.Cu at (116.3, 100.3)
- added REF**: SolderWirePad_1x01_SMD_1x2mm, Connector_Wire:SolderWirePad_1x01_SMD_1x2mm, F.Cu at (175.5, 96.5)
- added REF**: SolderWirePad_1x01_SMD_1x2mm, Connector_Wire:SolderWirePad_1x01_SMD_1x2mm, F.Cu at (116.3, 106.2)
- added REF**: SolderWirePad_1x01_SMD_1x2mm, Connector_Wire:SolderWirePad_1x01_SMD_1x2mm, B.Cu at (173.0, 87.6)
- added REF**: SolderWirePad_1x01_SMD_1x2mm, Connector_Wire:SolderWirePad_1x01_SMD_1x2mm, B.Cu at (119.9, 65.0)
- added REF**: SolderWirePad_1x01_SMD_1x2mm, Connector_Wire:SolderWirePad_1x01_SMD_1x2mm, B.Cu at (115.3, 137.7)
- added REF**: SolderWirePad_1x01_SMD_1x2mm, Connector_Wire:SolderWirePad_1x01_SMD_1x2mm, B.Cu at (125.0, 77.7)
- added REF**: SolderWirePad_1x01_SMD_1x2mm, Connector_Wire:SolderWirePad_1x01_SMD_1x2mm, B.Cu at (150.4, 54.4)
- added REF**: SolderWirePad_1x01_SMD_1x2mm, Connector_Wire:SolderWirePad_1x01_SMD_1x2mm, B.Cu at (111.0, 137.7)
- C2: footprint Capacitor_THT:C_Disc_D3.0mm_W1.6mm_P2.50mm -> Capacitor_THT:C_Disc_D4.3mm_W1.9mm_P5.00mm
- moved RFID1 125.5 mm to (1.52, 1.52), turned to 0 degrees
- moved U2 3.37 mm to (173.5, 68.1)
- moved U3 2.83 mm to (109.5, 75.7)
- moved R1 1.57 mm to (97.3, 116.6)
Connections:
- IC2 pad 6: LOCKER_1 -> LOCKER_2
- IC2 pad 7: LOCKER_2 -> unconnected-(IC2-QH_1-Pad7)
- IC2 pad 9: unconnected-(IC2-QH_2-Pad9) -> LOCKER_1
- SDOOR_1 pad 2: +3.3V -> GND
- SDOOR_2 pad 2: +3.3V -> GND
- U1 pad 15: DS -> SH_CP
- U1 pad 16: Net-(U1-EN) -> unconnected-(U1-EN-Pad16)
- U1 pad 8: ST_CP -> DS
- U1 pad 9: SH_CP -> ST_CP
Routing:
- net GND: track 201.6 -> 350.4 mm
- net Net-(U1-EN): track 61.2 -> 0.00 mm
- net +3.3V: track 133.0 -> 81.9 mm
- net +12V: track 66.8 -> 104.4 mm
- net Net-(D2-A): track 10.4 -> 25.2 mm
- net DS: track 21.0 -> 6.87 mm
- net Net-(D1-A): track 10.3 -> 21.3 mm
- net +5V: track 214.5 -> 224.6 mm
- net LOCKER_1: track 54.0 -> 44.0 mm
- net SDOOR2: track 48.5 -> 55.9 mm
- net Net-(LED-RGB-2.2-Pin_1): track 18.0 -> 14.6 mm
- net GREEN-LED: track 9.30 -> 12.8 mm
- net BLUE-LED: track 9.30 -> 12.8 mm
- net RED-LED-2: track 8.27 -> 11.7 mm
- net RED-LED: track 8.27 -> 11.7 mm
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Other:
- board text added: "IC2"
