File: pcb/kratos-pcb/fan_system.kicad_sch (KiCad schematic)
At the start: 3 parts, among them Q1 2N2222A

Commit message: ### added
Parts:
- added R3, R9: R, symbol Device:R
Connections:
- net +5V: now also R3.1; no longer Q1.3
- net FAN_PWM: now also R9.1; no longer Q1.2
- new net: Q1.3, R3.2
- new net: Q1.2, R9.2
Other:
- moved on the sheet: D1, Q1

Commit message: ### update     - kicad schematic
Parts:
- removed D1: D, Diode_THT:D_DO-34_SOD68_P7.62mm_Horizontal, symbol Device:D
- removed Q1: 2N2222A, 2N2222A:TO92254P470H750-3, symbol 2N2222A:2N2222A
- removed R3, R9: R, symbol Device:R
- FAN1: footprint Connector_PinHeader_2.00mm:PinHeader_1x02_P2.00mm_Vertical -> TerminalBlock:TerminalBlock_bornier-2_P5.08mm
Connections:
- net FAN_PWM: now also FAN1.1 (+)
Other:
- moved on the sheet: FAN1

Commit message: kicad
Connections:
- net GND is gone; now on net FAN_PWM: FAN1.2 (-)
- net FAN_PWM: no longer FAN1.1 (+)
- new net VCC: FAN1.1 (+)
Changed lines of the file:
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@@
+    (stroke (width 0) (type default))
+  )
+  (wire (pts (xy 97.79 90.17) (xy 101.6 90.17))
     (stroke (width 0) (type default))
   )
@@
     (stroke (width 0) (type default))
   )
-  (global_label "FAN_PWM" (shape input) (at 101.6 68.58 90) (fields_autoplaced)
-    (effects (font (size 1.27 1.27)) (justify left))
-    (property "Intersheetrefs" "${INTERSHEET_REFS}" (at 101.6 56.9467 90)
-      (effects (font (size 1.27 1.27)) (justify left) hide)
-    )
-  )
-  (symbol (lib_id "power:GND") (at 101.6 90.17 0) (unit 1)
-    (in_bom yes) (on_board yes) (dnp no) (fields_autoplaced)
-    (property "Reference" "#PWR08" (at 101.6 96.52 0)
-      (effects (font (size 1.27 1.27)) hide)
-    )
-    (property "Value" "GND" (at 101.6 95.25 0)
-      (effects (font (size 1.27 1.27)))
-    )
-    (property "Footprint" "" (at 101.6 90.17 0)
-      (effects (font (size 1.27 1.27)) hide)
-    )
-    (property "Datasheet" "" (at 101.6 90.17 0)
-      (effects (font (size 1.27 1.27)) hide)
-    )
-    (pin "1")
-    (instances
-      (project "kratos-pcb"
-        (path "/12f1b997-8c5f-4ef7-b036-7873ddaba48e/40f2ff16-84bd-4283-bb2c-5258389cef5b"
-          (reference "#PWR08") (unit 1)
-        )
-      )
+  (global_label "FAN_PWM" (shape input) (at 97.79 90.17 180) (fields_autoplaced)
+    (effects (font (size 1.27 1.27)) (justify right))
+    (property "Intersheetrefs" "${INTERSHEET_REFS}" (at 86.1567 90.17 0)
+      (effects (font (size 1.27 1.27)) (justify right) hide)
     )
   )
@@
         )
       )
+    )
+  )
+  (symbol (lib_id "power:VCC") (at 101.6 68.58 0) (unit 1)
+    (in_bom yes) (on_board yes) (dnp no) (fields_autoplaced)
+    (property "Reference" "#PWR08" (at 101.6 72.39 0)
+      (effects (font (size 1.27 1.27)) hide)
+    )
+    (property "Value" "VCC" (at 101.6 63.5 0)
+      (effects (font (size 1.27 1.27)))
+    )
+    (property "Footprint" "" (at 101.6 68.58 0)
+      (effects (font (size 1.27 1.27)) hide)
+    )
+    (property "Datasheet" "" (at 101.6 68.58 0)
+      (effects (font (size 1.27 1.27)) hide)
+    )
+    (pin "1")
+    (instances
+      (project "kratos-pcb"
+        (path "/12f1b997-8c5f-4ef7-b036-7873ddaba48e/40f2ff16-84bd-4283-bb2c-5258389cef5b"
+          (reference "#PWR08") (unit 1)
+        )
+      )

Commit message: ### added
Connections:
- net VCC renamed +5V
Changed lines of the file:
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@@
     )
   )
-  (symbol (lib_id "power:VCC") (at 101.6 68.58 0) (unit 1)
+  (symbol (lib_id "power:+5V") (at 101.6 68.58 0) (unit 1)
     (in_bom yes) (on_board yes) (dnp no) (fields_autoplaced)
     (property "Reference" "#PWR08" (at 101.6 72.39 0)
       (effects (font (size 1.27 1.27)) hide)
     )
-    (property "Value" "VCC" (at 101.6 63.5 0)
+    (property "Value" "+5V" (at 101.6 63.5 0)
       (effects (font (size 1.27 1.27)))
     )
