File: pcb/kratos-pcb/door_sensor.kicad_sch (KiCad schematic)
At the start: 2 parts

Commit message: ### added
Connections:
- net +3.3V: now reaches SDOOR_2.1 (Pin_1)
- net +3.3V: now also SDOOR_1.1 (Pin_1)
- net SDOOR2: now reaches SDOOR_2.2 (Pin_2)
- net SDOOR1: now reaches SDOOR_1.2 (Pin_2)
Other:
- moved on the sheet: SDOOR_1, SDOOR_2
Changed lines of the file:
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@@
 (kicad_sch (version 20230121) (generator eeschema)
   (paper "A4")
-  (symbol (lib_id "Connector:Conn_01x02_Pin") (at 48.26 49.53 180) (unit 1)
+  (junction (at 130.81 82.55) (diameter 0) (color 0 0 0 0)
+  )
+  (wire (pts (xy 130.81 82.55) (xy 130.81 93.98))
+    (stroke (width 0) (type default))
+  )
+  (wire (pts (xy 130.81 93.98) (xy 147.32 93.98))
+    (stroke (width 0) (type default))
+  )
+  (wire (pts (xy 130.81 82.55) (xy 146.05 82.55))
+    (stroke (width 0) (type default))
+  )
+  (wire (pts (xy 143.51 80.01) (xy 146.05 80.01))
+    (stroke (width 0) (type default))
+  )
+  (wire (pts (xy 143.51 91.44) (xy 147.32 91.44))
+    (stroke (width 0) (type default))
+  )
+  (wire (pts (xy 130.81 73.66) (xy 130.81 82.55))
+    (stroke (width 0) (type default))
+  )
+  (global_label "SDOOR2" (shape input) (at 143.51 91.44 180) (fields_autoplaced)
+    (effects (font (size 1.27 1.27)) (justify right))
+    (property "Intersheetrefs" "${INTERSHEET_REFS}" (at 132.9048 91.44 0)
+      (effects (font (size 1.27 1.27)) (justify right) hide)
+    )
+  )
+  (global_label "SDOOR1" (shape input) (at 143.51 80.01 180) (fields_autoplaced)
+    (effects (font (size 1.27 1.27)) (justify right))
+    (property "Intersheetrefs" "${INTERSHEET_REFS}" (at 132.9048 80.01 0)
+      (effects (font (size 1.27 1.27)) (justify right) hide)
+    )
+  )
+  (symbol (lib_id "Connector:Conn_01x02_Pin") (at 152.4 93.98 180) (unit 1)
     (in_bom yes) (on_board yes) (dnp no) (fields_autoplaced)
-    (property "Reference" "SDOOR_2" (at 47.625 54.61 0)
+    (property "Reference" "SDOOR_2" (at 151.765 99.06 0)
       (effects (font (size 1.27 1.27)))
     )
-    (property "Value" "Conn_01x02_Pin" (at 47.625 52.07 0)
+    (property "Value" "Conn_01x02_Pin" (at 151.765 96.52 0)
       (effects (font (size 1.27 1.27)))
     )
-    (property "Footprint" "Connector_PinSocket_2.00mm:PinSocket_1x02_P2.00mm_Vertical" (at 48.26 49.53 0)
+    (property "Footprint" "Connector_PinSocket_2.00mm:PinSocket_1x02_P2.00mm_Vertical" (at 152.4 93.98 0)
       (effects (font (size 1.27 1.27)) hide)
     )
-    (property "Datasheet" "~" (at 48.26 49.53 0)
+    (property "Datasheet" "~" (at 152.4 93.98 0)
       (effects (font (size 1.27 1.27)) hide)
     )
@@
     )
   )
-  (symbol (lib_id "Connector:Conn_01x02_Pin") (at 48.26 38.1 180) (unit 1)
-    (in_bom yes) (on_board yes) (dnp no)
-    (property "Reference" "SDOOR_1" (at 47.625 43.18 0)
+  (symbol (lib_id "power:+3.3V") (at 130.81 73.66 0) (unit 1)
+    (in_bom yes) (on_board yes) (dnp no) (fields_autoplaced)
+    (property "Reference" "#PWR015" (at 130.81 77.47 0)
+      (effects (font (size 1.27 1.27)) hide)
+    )
+    (property "Value" "+3.3V" (at 130.81 68.58 0)
       (effects (font (size 1.27 1.27)))
     )
-    (property "Value" "Conn_01x02_Pin" (at 47.625 40.64 0)
+    (property "Footprint" "" (at 130.81 73.66 0)
+      (effects (font (size 1.27 1.27)) hide)
+    )
+    (property "Datasheet" "" (at 130.81 73.66 0)
+      (effects (font (size 1.27 1.27)) hide)
+    )
+    (pin "1")
+    (instances
+      (project "kratos-pcb"
+        (path "/12f1b997-8c5f-4ef7-b036-7873ddaba48e/4443c0c9-e781-4ba2-81ba-b0b59780290a"
+          (reference "#PWR015") (unit 1)
+        )
+      )
+    )
+  )
+  (symbol (lib_id "Connector:Conn_01x02_Pin") (at 151.13 82.55 180) (unit 1)
+    (in_bom yes) (on_board yes) (dnp no)
+    (property "Reference" "SDOOR_1" (at 150.495 87.63 0)
       (effects (font (size 1.27 1.27)))
     )
-    (property "Footprint" "Connector_PinSocket_2.00mm:PinSocket_1x02_P2.00mm_Vertical" (at 48.26 38.1 0)
+    (property "Value" "Conn_01x02_Pin" (at 150.495 85.09 0)
+      (effects (font (size 1.27 1.27)))
+    )
+    (property "Footprint" "Connector_PinSocket_2.00mm:PinSocket_1x02_P2.00mm_Vertical" (at 151.13 82.55 0)
       (effects (font (size 1.27 1.27)) hide)
     )
-    (property "Datasheet" "~" (at 48.26 38.1 0)
+    (property "Datasheet" "~" (at 151.13 82.55 0)
       (effects (font (size 1.27 1.27)) hide)
     )

Commit message: ### update     - kicad schematic
Parts:
- removed SDOOR_1, SDOOR_2: Conn_01x02_Pin, Connector_PinSocket_2.00mm:PinSocket_1x02_P2.00mm_Vertical, symbol Connector:Conn_01x02_Pin
- added SDOOR_1, SDOOR_2: Screw_Terminal_01x02, TerminalBlock:TerminalBlock_bornier-2_P5.08mm, symbol Connector:Screw_Terminal_01x02
Connections:
- net +3.3V: now also SDOOR_1.2 (Pin_2), SDOOR_2.2 (Pin_2)
- net SDOOR1: now also SDOOR_1.1 (Pin_1)
- net SDOOR2: now also SDOOR_2.1 (Pin_1)
Changed lines of the file:
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@@
     (stroke (width 0) (type default))
   )
-  (wire (pts (xy 130.81 82.55) (xy 146.05 82.55))
+  (wire (pts (xy 143.51 80.01) (xy 147.32 80.01))
     (stroke (width 0) (type default))
   )
-  (wire (pts (xy 143.51 80.01) (xy 146.05 80.01))
+  (wire (pts (xy 130.81 82.55) (xy 147.32 82.55))
     (stroke (width 0) (type default))
   )
@@
     (property "Intersheetrefs" "${INTERSHEET_REFS}" (at 132.9048 80.01 0)
       (effects (font (size 1.27 1.27)) (justify right) hide)
-    )
-  )
-  (symbol (lib_id "Connector:Conn_01x02_Pin") (at 152.4 93.98 180) (unit 1)
-    (in_bom yes) (on_board yes) (dnp no) (fields_autoplaced)
-    (property "Reference" "SDOOR_2" (at 151.765 99.06 0)
-      (effects (font (size 1.27 1.27)))
-    )
-    (property "Value" "Conn_01x02_Pin" (at 151.765 96.52 0)
-      (effects (font (size 1.27 1.27)))
-    )
-    (property "Footprint" "Connector_PinSocket_2.00mm:PinSocket_1x02_P2.00mm_Vertical" (at 152.4 93.98 0)
-      (effects (font (size 1.27 1.27)) hide)
-    )
-    (property "Datasheet" "~" (at 152.4 93.98 0)
-      (effects (font (size 1.27 1.27)) hide)
-    )
-    (pin "1")
-    (pin "2")
-    (instances
-      (project "kratos-pcb"
-        (path "/12f1b997-8c5f-4ef7-b036-7873ddaba48e/4443c0c9-e781-4ba2-81ba-b0b59780290a"
-          (reference "SDOOR_2") (unit 1)
-        )
-      )
     )
   )
@@
     )
   )
-  (symbol (lib_id "Connector:Conn_01x02_Pin") (at 151.13 82.55 180) (unit 1)
-    (in_bom yes) (on_board yes) (dnp no)
-    (property "Reference" "SDOOR_1" (at 150.495 87.63 0)
-      (effects (font (size 1.27 1.27)))
+  (symbol (lib_id "Connector:Screw_Terminal_01x02") (at 152.4 80.01 0) (unit 1)
+    (in_bom yes) (on_board yes) (dnp no) (fields_autoplaced)
+    (property "Reference" "SDOOR_1" (at 154.94 80.01 0)
+      (effects (font (size 1.27 1.27)) (justify left))
     )
-    (property "Value" "Conn_01x02_Pin" (at 150.495 85.09 0)
-      (effects (font (size 1.27 1.27)))
+    (property "Value" "Screw_Terminal_01x02" (at 154.94 82.55 0)
+      (effects (font (size 1.27 1.27)) (justify left))
     )
-    (property "Footprint" "Connector_PinSocket_2.00mm:PinSocket_1x02_P2.00mm_Vertical" (at 151.13 82.55 0)
+    (property "Footprint" "TerminalBlock:TerminalBlock_bornier-2_P5.08mm" (at 152.4 80.01 0)
       (effects (font (size 1.27 1.27)) hide)
     )
-    (property "Datasheet" "~" (at 151.13 82.55 0)
+    (property "Datasheet" "~" (at 152.4 80.01 0)
       (effects (font (size 1.27 1.27)) hide)
     )
+    (pin "2")
     (pin "1")
-    (pin "2")
     (instances
       (project "kratos-pcb"
@@
         )
       )
+    )
+  )
+  (symbol (lib_id "Connector:Screw_Terminal_01x02") (at 152.4 91.44 0) (unit 1)
+    (in_bom yes) (on_board yes) (dnp no) (fields_autoplaced)
+    (property "Reference" "SDOOR_2" (at 154.94 91.44 0)
+      (effects (font (size 1.27 1.27)) (justify left))
+    )
+    (property "Value" "Screw_Terminal_01x02" (at 154.94 93.98 0)
+      (effects (font (size 1.27 1.27)) (justify left))
+    )
+    (property "Footprint" "TerminalBlock:TerminalBlock_bornier-2_P5.08mm" (at 152.4 91.44 0)
+      (effects (font (size 1.27 1.27)) hide)
+    )
+    (property "Datasheet" "~" (at 152.4 91.44 0)
+      (effects (font (size 1.27 1.27)) hide)
+    )
+    (pin "2")
+    (pin "1")
+    (instances
+      (project "kratos-pcb"
+        (path "/12f1b997-8c5f-4ef7-b036-7873ddaba48e/4443c0c9-e781-4ba2-81ba-b0b59780290a"
+          (reference "SDOOR_2") (unit 1)
+        )
+      )

Commit message: ### Modify
   - schematic
Parts:
- added R3, R4: 10k, Resistor_THT:R_Axial_DIN0207_L6.3mm_D2.5mm_P10.16mm_Horizontal, symbol Device:R
Connections:
- net +3.3V: now also R3.1, R4.1; no longer SDOOR_1.2 (Pin_2), SDOOR_2.2 (Pin_2)
- net SDOOR1: now also R3.2
- net SDOOR2: now also R4.2
- new net GND: SDOOR_1.2 (Pin_2), SDOOR_2.2 (Pin_2)
Changed lines of the file:
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@@
 (kicad_sch (version 20230121) (generator eeschema)
   (paper "A4")
-  (junction (at 130.81 82.55) (diameter 0) (color 0 0 0 0)
-  )
-  (wire (pts (xy 130.81 82.55) (xy 130.81 93.98))
-    (stroke (width 0) (type default))
-  )
-  (wire (pts (xy 130.81 93.98) (xy 147.32 93.98))
-    (stroke (width 0) (type default))
-  )
-  (wire (pts (xy 143.51 80.01) (xy 147.32 80.01))
-    (stroke (width 0) (type default))
-  )
-  (wire (pts (xy 130.81 82.55) (xy 147.32 82.55))
-    (stroke (width 0) (type default))
-  )
-  (wire (pts (xy 143.51 91.44) (xy 147.32 91.44))
-    (stroke (width 0) (type default))
-  )
-  (wire (pts (xy 130.81 73.66) (xy 130.81 82.55))
+  (junction (at 144.78 91.44) (diameter 0) (color 0 0 0 0)
+  )
+  (junction (at 130.81 76.2) (diameter 0) (color 0 0 0 0)
+  )
+  (junction (at 144.78 80.01) (diameter 0) (color 0 0 0 0)
+  )
+  (wire (pts (xy 147.32 93.98) (xy 144.78 93.98))
+    (stroke (width 0) (type default))
+  )
+  (wire (pts (xy 147.32 82.55) (xy 146.05 82.55))
+    (stroke (width 0) (type default))
+  )
+  (wire (pts (xy 144.78 76.2) (xy 144.78 80.01))
+    (stroke (width 0) (type default))
+  )
+  (wire (pts (xy 142.24 86.36) (xy 144.78 86.36))
+    (stroke (width 0) (type default))
+  )
+  (wire (pts (xy 143.51 80.01) (xy 144.78 80.01))
+    (stroke (width 0) (type default))
+  )
+  (wire (pts (xy 142.24 76.2) (xy 144.78 76.2))
+    (stroke (width 0) (type default))
+  )
+  (wire (pts (xy 144.78 93.98) (xy 144.78 95.25))
+    (stroke (width 0) (type default))
+  )
+  (wire (pts (xy 143.51 91.44) (xy 144.78 91.44))
+    (stroke (width 0) (type default))
+  )
+  (wire (pts (xy 130.81 86.36) (xy 134.62 86.36))
+    (stroke (width 0) (type default))
+  )
+  (wire (pts (xy 130.81 76.2) (xy 134.62 76.2))
+    (stroke (width 0) (type default))
+  )
+  (wire (pts (xy 144.78 80.01) (xy 147.32 80.01))
+    (stroke (width 0) (type default))
+  )
+  (wire (pts (xy 130.81 73.66) (xy 130.81 76.2))
+    (stroke (width 0) (type default))
+  )
+  (wire (pts (xy 146.05 82.55) (xy 146.05 83.82))
+    (stroke (width 0) (type default))
+  )
+  (wire (pts (xy 144.78 86.36) (xy 144.78 91.44))
+    (stroke (width 0) (type default))
+  )
+  (wire (pts (xy 130.81 76.2) (xy 130.81 86.36))
+    (stroke (width 0) (type default))
+  )
+  (wire (pts (xy 144.78 91.44) (xy 147.32 91.44))
     (stroke (width 0) (type default))
   )
@@
     )
   )
+  (symbol (lib_id "power:GND") (at 144.78 95.25 0) (unit 1)
+    (in_bom yes) (on_board yes) (dnp no)
+    (property "Reference" "#PWR09" (at 144.78 101.6 0)
+      (effects (font (size 1.27 1.27)) hide)
+    )
+    (property "Value" "GND" (at 147.32 99.06 0)
+      (effects (font (size 1.27 1.27)))
+    )
+    (property "Footprint" "" (at 144.78 95.25 0)
+      (effects (font (size 1.27 1.27)) hide)
+    )
+    (property "Datasheet" "" (at 144.78 95.25 0)
+      (effects (font (size 1.27 1.27)) hide)
+    )
+    (pin "1")
+    (instances
+      (project "kratos-pcb"
+        (path "/12f1b997-8c5f-4ef7-b036-7873ddaba48e/4443c0c9-e781-4ba2-81ba-b0b59780290a"
+          (reference "#PWR09") (unit 1)
+        )
+      )
+    )
+  )
+  (symbol (lib_id "Device:R") (at 138.43 76.2 90) (unit 1)
+    (in_bom yes) (on_board yes) (dnp no)
+    (property "Reference" "R3" (at 138.43 71.12 90)
+      (effects (font (size 1.27 1.27)))
+    )
+    (property "Value" "10k" (at 138.43 73.66 90)
+      (effects (font (size 1.27 1.27)))
+    )
+    (property "Footprint" "Resistor_THT:R_Axial_DIN0207_L6.3mm_D2.5mm_P10.16mm_Horizontal" (at 138.43 77.978 90)
+      (effects (font (size 1.27 1.27)) hide)
+    )
+    (property "Datasheet" "~" (at 138.43 76.2 0)
+      (effects (font (size 1.27 1.27)) hide)
+    )
+    (pin "1")
+    (pin "2")
+    (instances
+      (project "kratos-pcb"
+        (path "/12f1b997-8c5f-4ef7-b036-7873ddaba48e/4443c0c9-e781-4ba2-81ba-b0b59780290a"
+          (reference "R3") (unit 1)
+        )
+      )
+    )
+  )
   (symbol (lib_id "Connector:Screw_Terminal_01x02") (at 152.4 80.01 0) (unit 1)
     (in_bom yes) (on_board yes) (dnp no) (fields_autoplaced)
@@
         )
       )
+    )
+  )
+  (symbol (lib_id "Device:R") (at 138.43 86.36 90) (unit 1)
+    (in_bom yes) (on_board yes) (dnp no)
+    (property "Reference" "R4" (at 138.43 82.55 90)
+      (effects (font (size 1.27 1.27)))
+    )
+    (property "Value" "10k" (at 138.43 88.9 90)
+      (effects (font (size 1.27 1.27)))
+    )
+    (property "Footprint" "Resistor_THT:R_Axial_DIN0207_L6.3mm_D2.5mm_P10.16mm_Horizontal" (at 138.43 88.138 90)
+      (effects (font (size 1.27 1.27)) hide)
+    )
+    (property "Datasheet" "~" (at 138.43 86.36 0)
+      (effects (font (size 1.27 1.27)) hide)
+    )
+    (pin "1")
+    (pin "2")
+    (instances
+      (project "kratos-pcb"
+        (path "/12f1b997-8c5f-4ef7-b036-7873ddaba48e/4443c0c9-e781-4ba2-81ba-b0b59780290a"
+          (reference "R4") (unit 1)
+        )
+      )
+    )
+  )
+  (symbol (lib_id "power:GND") (at 146.05 83.82 0) (unit 1)
+    (in_bom yes) (on_board yes) (dnp no)
+    (property "Reference" "#PWR029" (at 146.05 90.17 0)
+      (effects (font (size 1.27 1.27)) hide)
+    )
+    (property "Value" "GND" (at 148.59 86.36 0)
+      (effects (font (size 1.27 1.27)))
+    )
+    (property "Footprint" "" (at 146.05 83.82 0)
+      (effects (font (size 1.27 1.27)) hide)
+    )
+    (property "Datasheet" "" (at 146.05 83.82 0)
+      (effects (font (size 1.27 1.27)) hide)
+    )
+    (pin "1")
+    (instances
+      (project "kratos-pcb"
+        (path "/12f1b997-8c5f-4ef7-b036-7873ddaba48e/4443c0c9-e781-4ba2-81ba-b0b59780290a"
+          (reference "#PWR029") (unit 1)
+        )
+      )
